Commit message: complete table

File: acc16model.xacro (robot description, xacro)
@@ -79,4 +79,5 @@
     </inertial>
   </link>
+  <!-- join right leg to base -->
   <joint name="base_to_right_leg" type="fixed">
     <parent link="base_link"/>
@@ -84,4 +85,5 @@
     <origin xyz="${(table_top_length/2)-0.0762} 0 0.3"/>
   </joint>
+<!-- draw left leg -->
   <link name="left_leg">
     <visual>
@@ -103,4 +105,5 @@
     </inertial>
   </link>
+  <!-- join left leg to base -->
   <joint name="base_to_left_leg" type="fixed">
     <parent link="base_link"/>
@@ -108,13 +111,13 @@
     <origin xyz="${-(table_top_length/2)+0.0762} 0 0.3"/>
   </joint>
-<!-- Table top -->
-<!--   <link name="table_top">
+<!-- Overlay table top -->
+  <link name="table_top">
     <visual>
-      <origin xyz="0 0 0" rpy="0 0 0" />
+      <origin xyz="0 0 ${table_leg_height}" rpy="0 0 0" />
       <geometry>
         <box size="${table_top_length} ${table_top_width} ${table_top_thickness}" />
       </geometry>
       <material name="table_color"/>
-      <origin xyz="0 0 0" rpy="0 0 0" />
+      <origin xyz="0 0 ${table_leg_height}" rpy="0 0 0" />
     </visual>
     <collision>
@@ -125,6 +128,16 @@
     <inertial>
       <mass value="10"/>
-      <inertia ixx="1.0" ixy="0.0" ixz="0.0" iyy="1.0" iyz="0.0" izz="1.0"/>
+       <inertia ixx="1.0" ixy="0.0" ixz="0.0" iyy="1.0" iyz="0.0" izz="1.0"/>
     </inertial>
-  </link> -->
+  </link>
+  <joint name="rightleg_to_tabletop" type="fixed">
+    <parent link="right_leg"/>
+    <child link="table_top" />
+    <origin xyz="${-(table_top_length/2)+0.0762} 0 -0.3 " />
+  </joint>
+  <joint name="leftleg_to_tabletop" type="fixed">
+    <parent link="left_leg"/>
+    <child link="table_top" />
+    <origin xyz="${-(table_top_length/2)+0.0762} 0 -0.3 " />
+  </joint>
 </robot>

Commit message: adjusted table-top origin

File: acc16model.xacro (robot description, xacro)
@@ -1,4 +1,4 @@
 <?xml version="1.0"?>
-<robot name="acctemp" xmlns:xacro="http://www.ros.org/wiki/xacro">
+<robot name="acc16model" xmlns:xacro="http://www.ros.org/wiki/xacro">
   <!-- Model for the Novalis Tx Spec
       Author: Olalekan Ogunmolu, August 2016
@@ -114,10 +114,10 @@
   <link name="table_top">
     <visual>
-      <origin xyz="0 0 ${table_leg_height}" rpy="0 0 0" />
+      <origin xyz="0 0 ${table_leg_height-0.65}" rpy="0 0 0" />
       <geometry>
         <box size="${table_top_length} ${table_top_width} ${table_top_thickness}" />
       </geometry>
       <material name="table_color"/>
-      <origin xyz="0 0 ${table_leg_height}" rpy="0 0 0" />
+      <origin xyz="0 0 ${table_leg_height-0.65}" rpy="0 0 0" />
     </visual>
     <collision>
@@ -134,10 +134,10 @@
     <parent link="right_leg"/>
     <child link="table_top" />
-    <origin xyz="${-(table_top_length/2)+0.0762} 0 -0.3 " />
+    <origin xyz="${-(table_top_length/2)+0.0762} 0 0.35 " />
   </joint>
   <joint name="leftleg_to_tabletop" type="fixed">
     <parent link="left_leg"/>
     <child link="table_top" />
-    <origin xyz="${-(table_top_length/2)+0.0762} 0 -0.3 " />
+    <origin xyz="${-(table_top_length/2)+0.0762} 0 0.35 " />
   </joint>
 </robot>

File: novalis.xacro (robot description, xacro)
@@ -1,4 +1,4 @@
 <?xml version="1.0"?>
-<robot name="acc2016_model" xmlns:xacro="http://www.ros.org/wiki/xacro">
+<robot name="novalis" xmlns:xacro="http://www.ros.org/wiki/xacro">
   <!-- Model for the Novalis Tx Spec
       Author: Olalekan Ogunmolu, August 2016
