Commit message: with stl file from adwait

File: bladder.xacro (robot description, xacro)
@@ -12,8 +12,7 @@
    <link name="bladder_link">
      <visual>
-       <origin xyz="0 0 0" rpy="0 0 ${-M_PI/2}" />
+       <origin xyz="0 0 0" rpy="0 0 0" />
        <geometry>
-         <box size="${bladder_length} ${bladder_width} ${bladder_thickness}" />
-         <!-- <mesh filename="package://superchick/meshes/bladder.STL" /> -->
+         <mesh filename="package://superchick/meshes/bladder.stl" scale=".001 .001 .001" />
        </geometry>
        <material name="bladder_color"/>
@@ -22,6 +21,5 @@
      <collision>
        <geometry>
-        <box size="${bladder_length} ${bladder_width} ${bladder_thickness}" />
-         <!-- <mesh filename="package://superchick/meshes/bladder.STL" /> -->
+         <mesh filename="package://superchick/meshes/bladder.stl" scale=".001 .001 .001" />
        </geometry>
      </collision>

File: superchick.xacro (robot description, xacro)
@@ -5,4 +5,6 @@
    <xacro:property name="head_width" value="0.2032" />
    <xacro:property name="head_thickness" value="0.1778" />
+   <xacro:property name="bladder_pos_x" value="-0.7" />
+   <xacro:property name="bladder_pos_y" value="-0.25" />
   <!-- This file contains the table and bladder descriptions -->
    <xacro:include filename="$(find superchick)/table.xacro" ns="table_ns" />
@@ -14,5 +16,5 @@
     <limit effort="200.0" lower="0.1016" upper="0.1016" velocity="1.0" />
     <safety_controller k_velocity="10" k_position="15" soft_lower_limit="-0.05" soft_upper_limit="0.05" />
-    <origin xyz="${-table_leg_posoffset-0.2} 0 0.05 " rpy="0 0 0" />
+    <origin xyz="${bladder_pos_x} ${bladder_pos_y} 0 " rpy="${M_PI/2} 0 ${M_PI/2}" />
    </joint>
 </robot>

File: table.xacro (robot description, xacro)
@@ -128,5 +128,5 @@
         <box size="${table_top_length} ${table_top_width} ${table_top_thickness}" />
       </geometry>
-      <material name="white"/>
+      <material name="table_color"/>
       <origin xyz="0 0 ${table_leg_height-0.65}" rpy="0 0 0" />
     </visual>
@@ -173,5 +173,5 @@
     <parent link="table_top"/>
     <child link="table_cover"/>
-    <origin xyz="0 ${(table_top_width/2)-0.1} -0.18" rpy="${-M_PI/2} 0 0 "/>
+    <origin xyz="0 ${(table_top_width/2)-0.08} -0.18" rpy="${-M_PI/2} 0 0 "/>
   </joint>
 </robot>
