Commit message: head and ball joint

File: whitehead.xacro (robot description, xacro)
@@ -16,5 +16,6 @@
        <origin xyz="${head_x_orig} ${head_y_orig} ${0}" rpy="0 0 0" />
        <geometry>
-         <mesh filename="package://superchick/meshes/white_head.stl" scale=".001 .001 .001" />
+         <mesh filename="package://superchick/meshes/headnball.STL" scale=".001 .001 .001" />
+         <!-- <mesh filename="package://superchick/meshes/white_head.stl" scale=".001 .001 .001" /> -->
        </geometry>
        <material name="brown"/>
@@ -23,5 +24,6 @@
      <collision>
        <geometry>
-         <mesh filename="package://superchick/meshes/white_head.stl" scale=".001 .001 .001" />
+         <mesh filename="package://superchick/meshes/headnball.STL" scale=".001 .001 .001" />
+         <!-- <mesh filename="package://superchick/meshes/white_head.stl" scale=".001 .001 .001" /> -->
        </geometry>
      </collision>
