Commit message: cleaned

File: superchick.xacro (robot description, xacro)
@@ -1,7 +1,12 @@
 <?xml version="1.0"?>
-<robot name="macroed" xmlns:xacro="http://ros.org/wiki/xacro">
-  <xacro:property name="width" value=".5" />
-  <xacro:property name="bodylen" value=".8" />
-  <xacro:property name="height" value=".1" />
+<!-- Olalekan Ogunmolu. June 2016. Model of the Novalis Tx  Radiosurgery Platform in ROS URDF -->
+<!--Ref 1: Novalis Tx
+            http://www.behestandarman.com/varian%20products/Delivery%20systems/Novalis/Novalis_Tx_Spec_10011B.pdf -->
+<!-- Ref 2: http://radonc.ucla.edu/novalis-tx -->
+<!-- Ref 3: https://www.novalis-radiosurgery.com/about-us/novalis-radiosurgery-family/ -->
+<robot name="superchicko" xmlns:xacro="http://ros.org/wiki/xacro">
+  <xacro:property name="width" value="${43.3*2}" />
+  <xacro:property name="bodylen" value="18.32" />
+  <xacro:property name="height" value="${25.84/2}" />
   <xacro:property name="wheeldiam" value=".07" />
   <xacro:property name="cyl_radius" value="2.1" />
@@ -34,5 +39,5 @@
         <box size="${width} ${bodylen} ${height}"/>
       </geometry>
-      <material name="gray" />
+      <material name="white" />
     </visual>
     <collision>

Commit message: finished 6-DOF bed frame

File: superchick.xacro (robot description, xacro)
@@ -5,5 +5,18 @@
 <!-- Ref 2: http://radonc.ucla.edu/novalis-tx -->
 <!-- Ref 3: https://www.novalis-radiosurgery.com/about-us/novalis-radiosurgery-family/ -->
-<robot name="superchicko" xmlns:xacro="http://ros.org/wiki/xacro">
+<robot name="superchick" xmlns:xacro="http://ros.org/wiki/xacro">
+  <!-- Macros -->
+  <xacro:macro name="material_color" params="name rgba">
+      <material name="${name}">
+          <color rgba="${rgba}" />
+      </material>
+  </xacro:macro>
+  <xacro:macro name="default_inertial" params="mass">
+    <inertial>
+      <mass value="${mass}" />
+      <inertia ixx="1.0" ixy="0.0" ixz="0.0" iyy="1.0" iyz="0.0" izz="1.0" />
+    </inertial>
+  </xacro:macro>
+   <xacro:include filename="novalis.macro.xacro" />
   <xacro:property name="width" value="${43.3*2}" />
   <xacro:property name="bodylen" value="18.32" />
@@ -13,4 +26,11 @@
   <xacro:property name="cyl_length" value="4.5" />
   <xacro:property name="pi" value="3.1415926535897931" />
+  <!-- Create the world link.
+      World is on the floor directly under the robot base
+      X points to the right when facing the robot
+      Y points toward the back of the robot
+      Z points up
+  -->
+  <link name="world" />
   <geometry type="cylinder" radius="${cyl_radius}" length="${cyl_length}" />
   <geometry type="box"      size="${width} ${bodylen} ${height}" />
@@ -28,10 +48,4 @@
     <color rgba="0.8 0.8 0.8 0.8"/>
   </material>
-  <xacro:macro name="default_inertial" params="mass">
-    <inertial>
-      <mass value="${mass}" />
-      <inertia ixx="1.0" ixy="0.0" ixz="0.0" iyy="1.0" iyz="0.0" izz="1.0" />
-    </inertial>
-  </xacro:macro>
   <link name="base_link">
     <visual>
@@ -48,126 +62,3 @@
     <xacro:default_inertial mass="10"/>
   </link>
-  <link name="bed_link">
-    <visual>
-      <geometry>
-        <box size="${width} ${bodylen} ${height}"/>
-      </geometry>
-      <origin rpy="0 0 0" xyz="0 0 -0.5"/>
-      <material name="blue"/>
-    </visual>
-    <collision>
-      <geometry>
-        <box size="${width} ${bodylen} ${height}"/>
-      </geometry>
-    </collision>
-  </link>
-  <joint name="base_to_bed" type="continuous">
-    <parent link="base_link"/>
-    <child link="bed_link"/>
-    <origin xyz="0 0 0.1"/>
-  </joint>
-  <!--Right Front of 6DOF Couch -->
-  <link name="right_front_wheel">
-    <visual>
-      <origin rpy="1.57075 0 0" xyz="0 0 0.1"/>
-      <geometry>
-        <cylinder length="0.1" radius="-0.035"/>
-      </geometry>
-      <material name="black"/>
-    </visual>
-    <collision>
-      <origin rpy="1.57075 0 0" xyz="0 0 0.1"/>
-      <geometry>
-        <cylinder length="0.1" radius="0.035"/>
-      </geometry>
-    </collision>
-    <inertial>
-      <mass value="1"/>
-      <inertia ixx="1.0" ixy="0.0" ixz="0.0" iyy="1.0" iyz="0.0" izz="1.0"/>
-    </inertial>
-  </link>
-  <joint name="right_front_wheel_joint" type="continuous">
-    <axis rpy="0 0 0" xyz="0 1 0"/>
-    <parent link="base_link"/>
-    <child link="right_front_wheel"/>
-    <origin rpy="0 0 0" xyz="0.133333333333 0 -0.45"/>
-  </joint>
-  <!--Right back wheel of 6 DOF couch -->
-  <link name="right_back_wheel">
-    <visual>
-      <origin rpy="1.57075 0 0" xyz="0 0 0.1"/>
-      <geometry>
-        <cylinder length="0.1" radius="0.035"/>
-      </geometry>
-      <material name="black"/>
-    </visual>
-    <collision>
-      <origin rpy="1.57075 0 0" xyz="0 0 0.1"/>
-      <geometry>
-        <cylinder length="0.1" radius="0.035"/>
-      </geometry>
-    </collision>
-    <inertial>
-      <mass value="1"/>
-      <inertia ixx="1.0" ixy="0.0" ixz="0.0" iyy="1.0" iyz="0.0" izz="1.0"/>
-    </inertial>
-  </link>
-  <joint name="right_back_wheel_joint" type="continuous">
-    <axis rpy="0 0 0" xyz="0 1 0"/>
-    <parent link="base_link"/>
-    <child link="right_back_wheel"/>
-    <origin rpy="0 0 0" xyz="-0.133333333333 0 -0.45"/>
-  </joint>
-  <!--Left Front of 6DOF Couch -->
-  <link name="left_front_wheel">
-    <visual>
-      <origin rpy="1.57075 0 0" xyz="-0.4 0.4 0.1"/>
-      <geometry>
-        <cylinder length="0.1" radius="-0.035"/>
-      </geometry>
-      <material name="black"/>
-    </visual>
-    <collision>
-      <origin rpy="1.57075 0 0" xyz="-0.4 0.4 0.1"/>
-      <geometry>
-        <cylinder length="0.1" radius="0.035"/>
-      </geometry>
-    </collision>
-    <inertial>
-      <mass value="1"/>
-      <inertia ixx="1.0" ixy="0.0" ixz="0.0" iyy="1.0" iyz="0.0" izz="1.0"/>
-    </inertial>
-  </link>
-  <joint name="left_front_wheel_joint" type="continuous">
-    <axis rpy="0 0 0" xyz="0 0.1 0"/>
-    <parent link="base_link"/>
-    <child link="left_front_wheel"/>
-    <origin rpy="0 0 0" xyz="0 0 -0.45"/>
-  </joint>
-  <!--Right back wheel of 6 DOF couch -->
-  <link name="left_back_wheel">
-    <visual>
-      <origin rpy="1.57075 0 0" xyz="0.4 0.4 0.1"/>
-      <geometry>
-        <cylinder length="0.1" radius="0.035"/>
-      </geometry>
-      <material name="black"/>
-    </visual>
-    <collision>
-      <origin rpy="1.57075 0 0" xyz="0.4 0.4 0.1"/>
-      <geometry>
-        <cylinder length="0.1" radius="0.035"/>
-      </geometry>
-    </collision>
-    <inertial>
-      <mass value="1"/>
-      <inertia ixx="1.0" ixy="0.0" ixz="0.0" iyy="1.0" iyz="0.0" izz="1.0"/>
-    </inertial>
-  </link>
-  <joint name="left_back_wheel_joint" type="continuous">
-    <axis rpy="0 0 0" xyz="0 1 0"/>
-    <parent link="base_link"/>
-    <child link="left_back_wheel"/>
-    <origin rpy="0 0 0" xyz="0 -0.133333333333 -0.45"/>
-  </joint>
 </robot>

Commit message: head height and bladder

File: superchick.xacro (robot description, xacro)
@@ -1,64 +1,36 @@
 <?xml version="1.0"?>
-<!-- Olalekan Ogunmolu. June 2016. Model of the Novalis Tx  Radiosurgery Platform in ROS URDF -->
-<!--Ref 1: Novalis Tx
-            http://www.behestandarman.com/varian%20products/Delivery%20systems/Novalis/Novalis_Tx_Spec_10011B.pdf -->
-<!-- Ref 2: http://radonc.ucla.edu/novalis-tx -->
-<!-- Ref 3: https://www.novalis-radiosurgery.com/about-us/novalis-radiosurgery-family/ -->
 <robot name="superchick" xmlns:xacro="http://ros.org/wiki/xacro">
-  <!-- Macros -->
-  <xacro:macro name="material_color" params="name rgba">
-      <material name="${name}">
-          <color rgba="${rgba}" />
-      </material>
-  </xacro:macro>
-  <xacro:macro name="default_inertial" params="mass">
-    <inertial>
-      <mass value="${mass}" />
-      <inertia ixx="1.0" ixy="0.0" ixz="0.0" iyy="1.0" iyz="0.0" izz="1.0" />
-    </inertial>
-  </xacro:macro>
-   <xacro:include filename="novalis.macro.xacro" />
-  <xacro:property name="width" value="${43.3*2}" />
-  <xacro:property name="bodylen" value="18.32" />
-  <xacro:property name="height" value="${25.84/2}" />
-  <xacro:property name="wheeldiam" value=".07" />
-  <xacro:property name="cyl_radius" value="2.1" />
-  <xacro:property name="cyl_length" value="4.5" />
-  <xacro:property name="pi" value="3.1415926535897931" />
-  <!-- Create the world link.
-      World is on the floor directly under the robot base
-      X points to the right when facing the robot
-      Y points toward the back of the robot
-      Z points up
-  -->
-  <link name="world" />
-  <geometry type="cylinder" radius="${cyl_radius}" length="${cyl_length}" />
-  <geometry type="box"      size="${width} ${bodylen} ${height}" />
-  <circle circumference="${2.5 * pi}" />
-  <material name="blue">
-    <color rgba="0 0 .8 1"/>
+   <!-- General Properties -->
+   <xacro:property name="bladder_length" value="0.4572" />
+   <xacro:property name="bladder_width" value="0.2794" />
+   <xacro:property name="bladder_thickness" value="0.1016" />
+   <xacro:property name="head_height" value="0.2794" />
+   <xacro:property name="head_width" value="0.2032" />
+   <xacro:property name="head_thickness" value="0.1778" />
+     <!-- Derived Variables -->
+  <material name="bladder_color" >
+    <color rgba="0.133333 0.545098 0.133333" /> <!--forest green-->
   </material>
-  <material name="black">
-    <color rgba="0 0 0 1"/>
-  </material>
-  <material name="white">
-    <color rgba="1 1 1 1"/>
-  </material>
-  <material name="gray">
-    <color rgba="0.8 0.8 0.8 0.8"/>
-  </material>
-  <link name="base_link">
-    <visual>
-      <geometry>
-        <box size="${width} ${bodylen} ${height}"/>
-      </geometry>
-      <material name="white" />
-    </visual>
-    <collision>
-      <geometry>
-        <box size="${width} ${bodylen} ${height}"/>
-      </geometry>
-    </collision>
-    <xacro:default_inertial mass="10"/>
-  </link>
+  <!-- This file contains the table description -->
+   <xacro:include filename="$(find superchick)/table.xacro" ns="table_ns" />
+   <!-- inflatable air bladder -->
+   <link name="bladder_link">
+     <visual>
+       <origin xyz="0 0 0" rpy="0 0 0" />
+       <geometry>
+         <box size="${table_top_length} ${table_top_width} ${table_top_thickness}" />
+       </geometry>
+       <material name="base_color"/>
+       <origin xyz="0 0 0" rpy="0 0 0" />
+     </visual>
+     <collision>
+       <geometry>
+         <box size="${table_top_length} ${table_top_width} ${table_top_thickness}" />
+       </geometry>
+     </collision>
+     <inertial>
+       <mass value="10"/>
+       <inertia ixx="1.0" ixy="0.0" ixz="0.0" iyy="1.0" iyz="0.0" izz="1.0"/>
+     </inertial>
+   </link>
 </robot>

File: table.xacro (robot description, xacro)
@@ -1,10 +1,10 @@
 <?xml version="1.0"?>
 <robot name="acc16model" xmlns:xacro="http://www.ros.org/wiki/xacro">
-  <!-- Model for the Novalis Tx Spec
+  <!-- Model for the Superchick Table Spec
       Author: Olalekan Ogunmolu, August 2016
         Generate urdf with
-        rosrun xacro xacro src/superchick/acc16model.xacro > acc16.urdf
+        rosrun xacro xacro src/superchick/table.xacro > table.urdf
         Then run with
-        roslaunch superchick display.launch model:=acc16.urdf
+        roslaunch superchick display.launch model:=table.urdf
   -->
   <!-- General Properties -->
@@ -39,4 +39,7 @@
     <color rgba="1 1 1 1"/>
   </material>
+  <material name="base_color">
+    <color rgba="0 0 0 0"/>
+  </material>
   <!-- table legs artificial base link -->
   <link name="base_link">
@@ -46,5 +49,5 @@
         <box size="${table_top_length} ${table_top_width} ${table_top_thickness}" />
       </geometry>
-      <material name="table_color"/>
+      <material name="base_color"/>
       <origin xyz="0 0 0" rpy="0 0 0" />
     </visual>
@@ -118,5 +121,5 @@
         <box size="${table_top_length} ${table_top_width} ${table_top_thickness}" />
       </geometry>
-      <material name="table_color"/>
+      <material name="white"/>
       <origin xyz="0 0 ${table_leg_height-0.65}" rpy="0 0 0" />
     </visual>

Commit message: table, bladder and pillow

File: superchick.xacro (robot description, xacro)
@@ -2,35 +2,17 @@
 <robot name="superchick" xmlns:xacro="http://ros.org/wiki/xacro">
    <!-- General Properties -->
-   <xacro:property name="bladder_length" value="0.4572" />
-   <xacro:property name="bladder_width" value="0.2794" />
-   <xacro:property name="bladder_thickness" value="0.1016" />
    <xacro:property name="head_height" value="0.2794" />
    <xacro:property name="head_width" value="0.2032" />
    <xacro:property name="head_thickness" value="0.1778" />
-     <!-- Derived Variables -->
-  <material name="bladder_color" >
-    <color rgba="0.133333 0.545098 0.133333" /> <!--forest green-->
-  </material>
-  <!-- This file contains the table description -->
+  <!-- This file contains the table and bladder descriptions -->
    <xacro:include filename="$(find superchick)/table.xacro" ns="table_ns" />
-   <!-- inflatable air bladder -->
-   <link name="bladder_link">
-     <visual>
-       <origin xyz="0 0 0" rpy="0 0 0" />
-       <geometry>
-         <box size="${table_top_length} ${table_top_width} ${table_top_thickness}" />
-       </geometry>
-       <material name="base_color"/>
-       <origin xyz="0 0 0" rpy="0 0 0" />
-     </visual>
-     <collision>
-       <geometry>
-         <box size="${table_top_length} ${table_top_width} ${table_top_thickness}" />
-       </geometry>
-     </collision>
-     <inertial>
-       <mass value="10"/>
-       <inertia ixx="1.0" ixy="0.0" ixz="0.0" iyy="1.0" iyz="0.0" izz="1.0"/>
-     </inertial>
-   </link>
+   <xacro:include filename="$(find superchick)/bladder.xacro" ns="bladder_ns" />
+   <!-- table link to bladder -->
+   <joint name="table_to_bladder" type="planar">
+    <parent link="table_top"/>
+    <child link="bladder_link"/>
+    <limit effort="200.0" lower="0.1016" upper="0.1016" velocity="1.0" />
+    <safety_controller k_velocity="10" k_position="15" soft_lower_limit="-0.05" soft_upper_limit="0.05" />
+    <origin xyz="${-table_leg_posoffset-0.2} 0 0.05 " rpy="0 0 0" />
+   </joint>
 </robot>

File: table.xacro (robot description, xacro)
@@ -26,4 +26,8 @@
   <!-- @TODO: not to scale distance between two legs -->
   <xacro:property name="legs_xdist" value="0.4" />
+  <!-- table cover properties -->
+  <xacro:property name="table_cover_length" value="1.524" />
+  <xacro:property name="table_cover_width" value="0.2794" />
+  <xacro:property name="table_cover_thickness" value="${0.127+0.1}" />
   <!-- Derived Variables -->
   <material name="table_color" >
@@ -33,6 +37,9 @@
     <color rgba="0 0 .8 1"/>
   </material>
-  <material name="black">
-    <color rgba="0 0 0 1"/>
+  <material name="table_cover_color">
+    <color rgba="0 ${26/255} ${51/255} 1"/>
+  </material>
+  <material name="dark_gray">
+    <color rgba="0.156863 0.156863 0.156863 1"/>
   </material>
   <material name="white">
@@ -69,5 +76,5 @@
       </geometry>
       <origin rpy="0 1.57075 0" xyz="0 0 0"/>
-      <material name="table_color"/>
+      <material name="dark_gray"/>
     </visual>
     <collision>
@@ -95,5 +102,5 @@
       </geometry>
       <origin rpy="0 1.57075 0" xyz="0 0 0"/>
-      <material name="table_color"/>
+      <material name="dark_gray"/>
     </visual>
     <collision>
@@ -144,3 +151,27 @@
     <origin xyz="${-(table_top_length/2)+0.0762} 0 0.35 " />
   </joint>
+  <link name="table_cover">
+    <visual>
+      <origin xyz="0 0 ${-table_top_thickness}" rpy="0 0 0" />
+      <geometry>
+        <box size="${table_cover_length} ${table_cover_width} ${table_cover_thickness}" />
+      </geometry>
+      <material name="table_cover_color"/>
+      <origin xyz="0 0 ${-table_top_thickness}" rpy="0 0 0" />
+    </visual>
+    <collision>
+      <geometry>
+        <box size="${table_cover_length} ${table_cover_width} ${table_cover_thickness}" />
+      </geometry>
+    </collision>
+    <inertial>
+      <mass value="10"/>
+       <inertia ixx="1.0" ixy="0.0" ixz="0.0" iyy="1.0" iyz="0.0" izz="1.0"/>
+    </inertial>
+  </link>
+  <joint name="tablecover_to_tabletop" type="fixed">
+    <parent link="table_top"/>
+    <child link="table_cover"/>
+    <origin xyz="0 ${(table_top_width/2)-0.1} -0.18" rpy="${-M_PI/2} 0 0 "/>
+  </joint>
 </robot>

Commit message: added stl head from kulkarni

File: superchick.xacro (robot description, xacro)
@@ -2,7 +2,4 @@
 <robot name="superchick" xmlns:xacro="http://ros.org/wiki/xacro">
    <!-- General Properties -->
-   <xacro:property name="head_height" value="0.2794" />
-   <xacro:property name="head_width" value="0.2032" />
-   <xacro:property name="head_thickness" value="0.1778" />
    <xacro:property name="bladder_pos_x" value="-0.7" />
    <xacro:property name="bladder_pos_y" value="-0.25" />
@@ -10,4 +7,5 @@
    <xacro:include filename="$(find superchick)/table.xacro" ns="table_ns" />
    <xacro:include filename="$(find superchick)/bladder.xacro" ns="bladder_ns" />
+   <xacro:include filename="$(find superchick)/whitehead.xacro" ns="whitehead_ns" />
    <!-- table link to bladder -->
    <joint name="table_to_bladder" type="planar">
@@ -18,3 +16,12 @@
     <origin xyz="${bladder_pos_x} ${bladder_pos_y} 0 " rpy="${M_PI/2} 0 ${M_PI/2}" />
    </joint>
+   <!-- bladder to whitehead -->
+   <joint name="bladder_to_whitehead" type="planar">
+    <parent link="bladder_link"/>
+    <child link="whitehead_link"/>
+    <limit effort="200.0" lower="0.1016" upper="0.1016" velocity="1.0" />
+    <safety_controller k_velocity="10" k_position="15" soft_lower_limit="-0.05" soft_upper_limit="0.05" />
+    <origin xyz="0.3 ${bladder_pos_y+0.35} 1.0" rpy="${-M_PI/2} 0 0" />
+   </joint>
 </robot>
+<!-- ${(table_top_length/2)-0.6} -->

Commit message: gead with ball

File: superchick.xacro (robot description, xacro)
@@ -7,5 +7,6 @@
    <xacro:include filename="$(find superchick)/table.xacro" ns="table_ns" />
    <xacro:include filename="$(find superchick)/bladder.xacro" ns="bladder_ns" />
-   <xacro:include filename="$(find superchick)/whitehead.xacro" ns="whitehead_ns" />
+   <!-- <xacro:include filename="$(find superchick)/whitehead.xacro" ns="whitehead_ns" /> -->
+   <xacro:include filename="$(find superchick)/headnball.xacro" ns="headnball_ns" />
    <!-- table link to bladder -->
    <joint name="table_to_bladder" type="planar">
@@ -17,5 +18,5 @@
    </joint>
    <!-- bladder to whitehead -->
-   <joint name="bladder_to_whitehead" type="planar">
+<!--    <joint name="bladder_to_whitehead" type="planar">
     <parent link="bladder_link"/>
     <child link="whitehead_link"/>
@@ -23,4 +24,11 @@
     <safety_controller k_velocity="10" k_position="15" soft_lower_limit="-0.05" soft_upper_limit="0.05" />
     <origin xyz="0.3 ${bladder_pos_y+0.35} 1.0" rpy="${-M_PI/2} 0 0" />
+   </joint> -->
+   <joint name="bladder_to_headnball" type="planar">
+    <parent link="bladder_link"/>
+    <child link="headnball_link"/>
+    <limit effort="200.0" lower="0.1016" upper="0.1016" velocity="1.0" />
+    <safety_controller k_velocity="10" k_position="15" soft_lower_limit="-0.05" soft_upper_limit="0.05" />
+    <origin xyz="0.3 ${bladder_pos_y+0.35} ${0.5}" rpy="${-M_PI/2} 0 0" />
    </joint>
 </robot>
