Commit message: move it configurations

File: headnball.xacro (robot description, xacro)
@@ -13,10 +13,10 @@
    <link name="headnball_link">
      <visual>
-       <origin xyz="${0} ${0} ${0}" rpy="${M_PI/2} 0 ${-M_PI}" />
+       <origin xyz="${0} ${0} ${-0.05}" rpy="${M_PI/2} 0 ${-M_PI}" />
        <geometry>
          <mesh filename="package://superchick/meshes/headnball.STL" scale=".001 .001 .001" />
        </geometry>
        <material name="brown"/>
-       <origin xyz="${0} ${0} ${0}" rpy="${M_PI/2} 0 ${-M_PI}" />
+       <origin xyz="${0} ${0} ${-0.05}" rpy="${M_PI/2} 0 ${-M_PI}" />
      </visual>
      <collision>
@@ -31,3 +31,2 @@
    </link>
 </robot>
-<!-- ${head_x_orig} ${head_y_orig-0.1} ${0} -->

File: superchick.xacro (robot description, xacro)
@@ -25,5 +25,5 @@
     <origin xyz="0.3 ${bladder_pos_y+0.35} 1.0" rpy="${-M_PI/2} 0 0" />
    </joint> -->
-   <joint name="bladder_to_headnball" type="planar">
+   <joint name="bladder_to_headnball" type="continuous">
     <parent link="bladder_link"/>
     <child link="headnball_link"/>
