Commit message: publishing joint states

File: superchick/headnball.xacro (robot description, xacro)
@@ -10,4 +10,10 @@
   <color rgba="0.647059 0.164706 0.164706 1"/>
   </material>
+  <!-- Used for fixing robot to Gazebo 'base_link' -->
+<!--     <link name="world"/>
+    <joint name="fixed" type="fixed">
+      <parent link="world"/>
+      <child link="headnball_link"/>
+    </joint> -->
    <!-- inflatable air bladder -->
    <link name="headnball_link">

File: superchick/superchick.xacro (robot description, xacro)
@@ -33,6 +33,6 @@
    </joint>
   <!-- Motion capture to base link -->
-  <joint name="motion_capture_to_base_link" type="fixed">
-    <parent link="base_link"/>
+  <joint name="motion_capture_to_world" type="fixed">
+    <parent link="world"/>
     <child link="motion_capture_frame"/>
     <origin xyz="-5 -4 2.54" rpy="0 0 0" />

File: superchick/table.xacro (robot description, xacro)
@@ -50,5 +50,5 @@
   </material>
   <!-- table legs artificial base link -->
-  <link name="base_link">
+  <link name="world">
     <visual>
       <origin xyz="0 0 0" rpy="0 0 0" />
@@ -64,8 +64,4 @@
       </geometry>
     </collision>
-<!--     <inertial>
-      <mass value="10"/>
-      <inertia ixx="1.0" ixy="0.0" ixz="0.0" iyy="1.0" iyz="0.0" izz="1.0"/>
-    </inertial> -->
   </link>
 <!-- right leg -->
@@ -85,11 +81,12 @@
     </collision>
     <inertial>
+      <origin xyz="0 0 0" rpy="0 0 0" />
       <mass value="10"/>
-      <inertia ixx="1.0" ixy="0.0" ixz="0.0" iyy="1.0" iyz="0.0" izz="1.0"/>
+      <inertia ixx="1e-1" ixy="0.0" ixz="0.0" iyy="1e-1" iyz="0.0" izz="1e-1"/>
     </inertial>
   </link>
   <!-- join right leg to base -->
   <joint name="base_to_right_leg" type="fixed">
-    <parent link="base_link"/>
+    <parent link="world"/>
     <child link="right_leg"/>
     <origin xyz="${(table_top_length/2)-0.0762} 0 0.3"/>
@@ -117,5 +114,5 @@
   <!-- join left leg to base -->
   <joint name="base_to_left_leg" type="fixed">
-    <parent link="base_link"/>
+    <parent link="world"/>
     <child link="left_leg"/>
     <origin xyz="${-(table_top_length/2)+0.0762} 0 0.3"/>
