Commit message: Alex's cage integration with Superchick

File: superchick/cage.xacro (robot description, xacro)
@@ -8,20 +8,21 @@
 	<!-- Panel Properties -->
 	<xacro:property name="side_panel_length" value=".231775" />
-	<xacro:property name="panel_12_oc_length" value=".34925" />
+	<xacro:property name="panel_12_oc_length" value=".4700" /> <!--.34925 -->
 	<xacro:property name="panel_height" value=".200025" />
 	<xacro:property name="panel_thickness" value=".0047625" />
-	<xacro:property name="base_link_length" value=".5842" />
-	<xacro:property name="base_link_width" value=".2794" />
-	<xacro:property name ="distance_panel_12_oc_from_center" value ="${(base_link_width/2) - .04572}" />
+	<xacro:property name="base_panel_length" value=".5842" />
+	<xacro:property name="base_panel_width" value=".2794" />
+	<xacro:property name ="distance_panel_12_oc_from_center" value ="${(base_panel_width/2) - .04572}" />
+	<!--<xacro:include filename="$(find superchick)/table.xacro" ns="table_ns" /> -->
 	<!-- Derived Variables -->
 	<material name="panel_color" >
-		<color rgba="0 100 0 1" />
+		<color rgba=".1 .1 .1 1" />
 	</material>
-	<!-- Base Link (Base Panel) -->
-	<link name="base_link">
+	<!-- Base panel -->
+	<link name="base_panel">
 		<visual>
 			<origin xyz="0 0 0" rpy="0 0 0" />
 			<geometry>
-				<box size="${base_link_length} ${base_link_width} ${panel_thickness}" />
+				<box size="${base_panel_length} ${base_panel_width} ${panel_thickness}" />
 			</geometry>
 			<material name="panel_color" />
@@ -30,8 +31,15 @@
 			<origin xyz="0 0 0" rpy="0 0 0" />
 			<geometry>
-				<box size="${base_link_length} ${base_link_width} ${panel_thickness}" />
+				<box size="${base_panel_length} ${base_panel_width} ${panel_thickness}" />
 			</geometry>
 		</collision>
 	</link>
+<!--
+	<joint name="base_panel_to_table_top" type="fixed">
+		<parent link="table_top"/>
+		<child link="base_panel"/>
+		<origin xyz="${cage_pos_x} ${cage_pos_y} ${(panel_thickness/2)}" rpy="0 0 ${PI/2}" />
+	</joint>
+-->
 	<!-- 12:00 panel -->
 	<link name="panel_12_oc">
@@ -50,7 +58,7 @@
 		</collision>
 	</link>
-	<!-- Join 12:00 Panel to Base -->
-	<joint name="panel_12_oc_to_base_link" type="fixed">
-		<parent link="base_link"/>
+	<!-- Join 12:00 Panel to base_panel -->
+	<joint name="panel_12_oc_to_base_panel" type="fixed">
+		<parent link="base_panel"/>
 		<child link="panel_12_oc"/>
 		<origin xyz="0 ${distance_panel_12_oc_from_center} ${(panel_thickness/2) + (panel_height/2)}" />

Commit message: Alex's final/revised integration of cage with Superchick

File: superchick/cage.xacro (robot description, xacro)
@@ -2,5 +2,5 @@
 <robot name="cage" xmlns:xacro="http://ros.org/wiki/xacro">
 	<!-- Description: A model of the "cage" used in the superchick project.
-	 Author: Alex Tomkovich, September 2016
+	 Author: Alex Tomkovich, September 27, 2016
  	-->
 	<!-- Constants -->
@@ -14,5 +14,4 @@
 	<xacro:property name="base_panel_width" value=".2794" />
 	<xacro:property name ="distance_panel_12_oc_from_center" value ="${(base_panel_width/2) - .04572}" />
-	<!--<xacro:include filename="$(find superchick)/table.xacro" ns="table_ns" /> -->
 	<!-- Derived Variables -->
 	<material name="panel_color" >
@@ -35,11 +34,4 @@
 		</collision>
 	</link>
-<!--
-	<joint name="base_panel_to_table_top" type="fixed">
-		<parent link="table_top"/>
-		<child link="base_panel"/>
-		<origin xyz="${cage_pos_x} ${cage_pos_y} ${(panel_thickness/2)}" rpy="0 0 ${PI/2}" />
-	</joint>
--->
 	<!-- 12:00 panel -->
 	<link name="panel_12_oc">

File: superchick/superchick.xacro (robot description, xacro)
@@ -9,6 +9,7 @@
    <!-- <xacro:include filename="$(find superchick)/whitehead.xacro" ns="whitehead_ns" /> -->
    <xacro:include filename="$(find superchick)/headnball.xacro" ns="headnball_ns" />
+   <xacro:include filename="$(find superchick)/cage.xacro" ns="cage_ns" />
    <!-- table link to bladder -->
-   <joint name="table_to_bladder" type="fixed">
+    <joint name="table_to_bladder" type="fixed">
     <parent link="table_top"/>
     <child link="bladder_link"/>
@@ -18,5 +19,6 @@
    </joint>
    <!-- bladder to whitehead -->
-<!--    <joint name="bladder_to_whitehead" type="planar">
+   <!--
+    <joint name="bladder_to_whitehead" type="planar">
     <parent link="bladder_link"/>
     <child link="whitehead_link"/>
@@ -25,4 +27,10 @@
     <origin xyz="0.3 ${bladder_pos_y+0.35} 1.0" rpy="${-M_PI/2} 0 0" />
    </joint> -->
+  <!-- base panel to table -->
+  <joint name="base_panel_to_table_top" type="fixed">
+    <parent link="table_top"/>
+    <child link="base_panel"/>
+    <origin xyz="${bladder_pos_x + .08} ${bladder_pos_y + .23} ${(panel_thickness/2)}" rpy="0 0 ${PI/2}" />
+  </joint>
    <joint name="bladder_to_headnball" type="continuous">
     <parent link="bladder_link"/>

Commit message: kinetic-master

File: superchick/cage.xacro (robot description, xacro)
@@ -5,5 +5,5 @@
  	-->
 	<!-- Constants -->
-	<xacro:property name="PI" value="3.14159" />
+	<xacro:property name="M_PI" value="3.14159" />
 	<!-- Panel Properties -->
 	<xacro:property name="side_panel_length" value=".231775" />
@@ -37,5 +37,5 @@
 	<link name="panel_12_oc">
 		<visual>
-			<origin xyz="0 0 0" rpy="${(PI/2)} 0 0" />
+			<origin xyz="0 0 0" rpy="${M_PI/2} 0 0" />
 			<geometry>
 				<box size="${panel_12_oc_length} ${panel_height} ${panel_thickness}" />
@@ -44,5 +44,5 @@
 		</visual>
 		<collision>
-			<origin xyz="0 0 0" rpy="${(PI/2)} 0 0" />
+			<origin xyz="0 0 0" rpy="${M_PI/2} 0 0" />
 			<geometry>
 				<box size="${panel_12_oc_length} ${panel_height} ${panel_thickness}" />
@@ -59,5 +59,5 @@
 	<link name="panel_9_oc">
 		<visual>
-			<origin xyz="0 0 0" rpy="${(PI/2)} 0 ${(PI/2)}" />
+			<origin xyz="0 0 0" rpy="${M_PI/2} 0 ${M_PI/2}" />
 			<geometry>
 				<box size="${side_panel_length} ${panel_height} ${panel_thickness}" />
@@ -66,5 +66,5 @@
 		</visual>
 		<collision>
-			<origin xyz="0 0 0" rpy="${(PI/2)} 0 ${(PI/2)}" />
+			<origin xyz="0 0 0" rpy="${M_PI/2} 0 ${M_PI/2}" />
 			<geometry>
 				<box size="${side_panel_length} ${panel_height} ${panel_thickness}" />
@@ -81,5 +81,5 @@
 	<link name="panel_3_oc">
 		<visual>
-			<origin xyz="0 0 0" rpy="${(PI/2)} 0 ${(PI/2)}" />
+			<origin xyz="0 0 0" rpy="${M_PI/2} 0 ${M_PI/2}" />
 			<geometry>
 				<box size="${side_panel_length} ${panel_height} ${panel_thickness}" />
@@ -88,5 +88,5 @@
 		</visual>
 		<collision>
-			<origin xyz="0 0 0" rpy="${(PI/2)} 0 ${(PI/2)}" />
+			<origin xyz="0 0 0" rpy="${M_PI/2} 0 ${M_PI/2}" />
 			<geometry>
 				<box size="${side_panel_length} ${panel_height} ${panel_thickness}" />

File: superchick/headnball.xacro (robot description, xacro)
@@ -5,4 +5,5 @@
    <xacro:property name="head_width" value="0.2032" />
    <xacro:property name="head_thickness" value="0.1778" />
+   <xacro:property name="M_PI" value="3.14159" />
   <xacro:property name="head_x_orig" value="-0.1" />
   <xacro:property name="head_y_orig" value="0.25" />

File: superchick/superchick.xacro (robot description, xacro)
@@ -1,4 +1,6 @@
 <?xml version="1.0"?>
 <robot name="superchick" xmlns:xacro="http://www.ros.org/wiki/xacro">
+  <!-- Constants -->
+  <xacro:property name="M_PI" value="3.14159" />
    <!-- General Properties -->
    <xacro:property name="bladder_pos_x" value="-0.7" />
@@ -23,5 +25,5 @@
     <parent link="table_top"/>
     <child link="base_panel"/>
-    <origin xyz="${bladder_pos_x + .08} ${bladder_pos_y + .23} ${(panel_thickness/2)}" rpy="0 0 ${PI/2}" />
+    <origin xyz="${bladder_pos_x + .08} ${bladder_pos_y + .23} ${cage_ns.panel_thickness/2}" rpy="0 0 ${M_PI/2}" />
   </joint>
    <joint name="bladder_to_headnball" type="continuous">

Commit message: updated head

File: superchick/cage.xacro (robot description, xacro)
@@ -1,6 +1,7 @@
 <?xml version="1.0"?>
 <robot name="cage" xmlns:xacro="http://www.ros.org/wiki/xacro">
-	<!-- Description: A model of the "cage" used in the superchick project.
+	<!-- Description: Head Cage
 	 Author: Alex Tomkovich, September 27, 2016
+	 Modified: Lekan Ogunmolu Nov. 18, 2016
  	-->
 	<!-- Constants -->
@@ -16,37 +17,47 @@
 	<!-- Derived Variables -->
 	<material name="panel_color" >
-		<color rgba=".1 .1 .1 1" />
+		<color rgba="0.133 0.55 0.13 1" />
 	</material>
 	<!-- Base panel -->
 	<link name="base_panel">
 		<visual>
-			<origin xyz="0 0 0" rpy="0 0 0" />
 			<geometry>
 				<box size="${base_panel_length} ${base_panel_width} ${panel_thickness}" />
 			</geometry>
+			<origin xyz="0 0 0" rpy="0 0 0" />
 			<material name="panel_color" />
 		</visual>
 		<collision>
-			<origin xyz="0 0 0" rpy="0 0 0" />
 			<geometry>
 				<box size="${base_panel_length} ${base_panel_width} ${panel_thickness}" />
 			</geometry>
+			<origin xyz="0 0 0" rpy="0 0 0" />
 		</collision>
+		<inertial>
+		  <origin xyz="0 0 0" rpy="0 0 0" />
+		  <mass value="0.1"/>
+		  <inertia ixx="1e-1" ixy="0.0" ixz="0.0" iyy="1e-1" iyz="0.0" izz="1e-1"/>
+		</inertial>
 	</link>
 	<!-- 12:00 panel -->
 	<link name="panel_12_oc">
 		<visual>
-			<origin xyz="0 0 0" rpy="${(PI/2)} 0 0" />
 			<geometry>
 				<box size="${panel_12_oc_length} ${panel_height} ${panel_thickness}" />
 			</geometry>
 			<material name="panel_color" />
+			<origin xyz="0 0 0" rpy="${(PI/2)} 0 0" />
 		</visual>
 		<collision>
-			<origin xyz="0 0 0" rpy="${(PI/2)} 0 0" />
 			<geometry>
 				<box size="${panel_12_oc_length} ${panel_height} ${panel_thickness}" />
 			</geometry>
+			<origin xyz="0 0 0" rpy="${(PI/2)} 0 0" />
 		</collision>
+		<inertial>
+		  <origin xyz="0 0 0" rpy="0 0 0" />
+		  <mass value="0.1"/>
+		  <inertia ixx="1e-1" ixy="0.0" ixz="0.0" iyy="1e-1" iyz="0.0" izz="1e-1"/>
+		</inertial>
 	</link>
 	<!-- Join 12:00 Panel to base_panel -->
@@ -66,9 +77,14 @@
 		</visual>
 		<collision>
-			<origin xyz="0 0 0" rpy="${(PI/2)} 0 ${(PI/2)}" />
 			<geometry>
 				<box size="${side_panel_length} ${panel_height} ${panel_thickness}" />
 			</geometry>
+			<origin xyz="0 0 0" rpy="${(PI/2)} 0 ${(PI/2)}" />
 		</collision>
+		<inertial>
+		  <origin xyz="0 0 0" rpy="0 0 0" />
+		  <mass value="0.1"/>
+		  <inertia ixx="1e-1" ixy="0.0" ixz="0.0" iyy="1e-1" iyz="0.0" izz="1e-1"/>
+		</inertial>
 	</link>
 	<!-- Join 9:00 Panel to 12:00 Panel -->
@@ -88,9 +104,14 @@
 		</visual>
 		<collision>
-			<origin xyz="0 0 0" rpy="${(PI/2)} 0 ${(PI/2)}" />
 			<geometry>
 				<box size="${side_panel_length} ${panel_height} ${panel_thickness}" />
 			</geometry>
+			<origin xyz="0 0 0" rpy="${(PI/2)} 0 ${(PI/2)}" />
 		</collision>
+		<inertial>
+		  <origin xyz="0 0 0" rpy="0 0 0" />
+		  <mass value="0.1"/>
+		  <inertia ixx="1e-1" ixy="0.0" ixz="0.0" iyy="1e-1" iyz="0.0" izz="1e-1"/>
+		</inertial>
 	</link>
 	<!-- Join 3:00 Panel to 12:00 Panel -->

File: superchick/headnball.xacro (robot description, xacro)
@@ -5,4 +5,5 @@
    <xacro:property name="head_width" value="0.2032" />
    <xacro:property name="head_thickness" value="0.1778" />
+   <xacro:property name="M_PI" value="3.14159" ns="headnball"/>
   <xacro:property name="head_x_orig" value="-0.1" />
   <xacro:property name="head_y_orig" value="0.25" />
@@ -10,10 +11,4 @@
   <color rgba="0.647059 0.164706 0.164706 1"/>
   </material>
-  <!-- Used for fixing robot to Gazebo 'base_link' -->
-<!--     <link name="world"/>
-    <joint name="fixed" type="fixed">
-      <parent link="world"/>
-      <child link="headnball_link"/>
-    </joint> -->
    <!-- inflatable air bladder -->
    <link name="headnball_link">
@@ -21,18 +16,38 @@
        <origin xyz="${0} ${0} ${-0.05}" rpy="${M_PI/2} 0 ${-M_PI}" />
        <geometry>
-         <mesh filename="package://superchick/meshes/headnball.STL" scale=".001 .001 .001" />
+         <mesh filename="package://superchick/meshes/headnball.dae" scale=".001 .001 .001" />
        </geometry>
        <material name="brown"/>
-       <origin xyz="${0} ${0} ${-0.05}" rpy="${M_PI/2} 0 ${-M_PI}" />
+       <origin xyz="${0} ${0} ${0}" rpy="${M_PI/2} 0 ${-M_PI}" />
      </visual>
      <collision>
        <geometry>
-         <mesh filename="package://superchick/meshes/headnball.STL" scale=".001 .001 .001" />
+         <mesh filename="package://superchick/meshes/headnball.dae" scale=".001 .001 .001" />
        </geometry>
+       <origin xyz="${0} ${0} ${0}" rpy="${M_PI/2} 0 ${-M_PI}" />
      </collision>
      <inertial>
-       <mass value="10"/>
-       <inertia ixx="1.0" ixy="0.0" ixz="0.0" iyy="1.0" iyz="0.0" izz="1.0"/>
+       <mass value="1e-1"/>
+       <inertia ixx="0.925288" ixy="0.379102" ixz="0.011081"
+                iyy="0.919140" iyz="0.111180" izz="0.993738"/>
      </inertial>
    </link>
 </robot>
+<!--
+Mesh Bounding Box Size 183.247528 233.881210 390.197662
+Mesh Bounding Box Diag 490.442963
+Mesh Volume is 1747609.625000
+Mesh Surface is 308892.718750
+Thin shell barycenter 95.753151 109.246353 218.224380
+Center of Mass is 98.803001 53.798462 504.412964
+Inertia Tensor is :
+| -213251981312.000000 -4579728384.000000 3054556928.000000 |
+| -4579728384.000000 -220260909056.000000 26342836224.000000 |
+| 3054556928.000000 26342836224.000000 11755722752.000000 |
+Principal axes are :
+| 0.925288 0.379102 0.011081 |
+| -0.377915 0.919140 0.111180 |
+| 0.031964 -0.107061 0.993738 |
+axis momenta are :
+| -211275972608.000000 -225218248704.000000 14737041408.000000 |
+ -->

File: superchick/superchick.xacro (robot description, xacro)
@@ -3,38 +3,64 @@
    <!-- General Properties -->
    <xacro:property name="bladder_pos_x" value="-0.7" />
-   <xacro:property name="bladder_pos_y" value="-0.25" />
+   <xacro:property name="bladder_pos_y" value="-0.35" />
   <!-- This file contains the table and bladder descriptions -->
    <xacro:include filename="$(find superchick)/table.xacro" ns="table_ns" />
-   <xacro:include filename="$(find superchick)/bladder.xacro" ns="bladder_ns" />
-   <!-- <xacro:include filename="$(find superchick)/whitehead.xacro" ns="whitehead_ns" /> -->
+   <xacro:include filename="$(find superchick)/bladders.xacro" ns="bladder_ns" />
    <xacro:include filename="$(find superchick)/headnball.xacro" ns="headnball_ns" />
    <xacro:include filename="$(find superchick)/cage.xacro" ns="cage_ns" />
-   <xacro:include filename="$(find superchick)/motionCaptureSystem.xacro" ns="motionCaptureSystem_ns" />
-   <!-- table link to bladder -->
-    <joint name="table_to_bladder" type="fixed">
+   <xacro:include filename="$(find superchick)/vicon.xacro" ns="vicon_ns" />
+   <!-- table link to bladders -->
+  <joint name="table_to_big_bladder" type="fixed">
     <parent link="table_top"/>
-    <child link="bladder_link"/>
+    <child link="big_bladder_link"/>
     <limit effort="200.0" lower="0.1016" upper="0.1016" velocity="1.0" />
     <safety_controller k_velocity="10" k_position="15" soft_lower_limit="-0.05" soft_upper_limit="0.05" />
-    <origin xyz="${bladder_pos_x} ${bladder_pos_y} 0 " rpy="${M_PI/2} 0 ${M_PI/2}" />
-   </joint>
-  <!-- base panel to table -->
-  <joint name="base_panel_to_table_top" type="fixed">
+    <origin xyz="${-(table_top_length)/2 + 0.2} 0 ${1e-1/3}" rpy="${0} 0 ${0}" />
+  </joint>
+  <joint name="table_to_rightneckbladder" type="fixed">
+    <parent link="table_top"/>
+    <child link="right_bladder"/>
+    <limit effort="200.0" lower="0.1016" upper="0.1016" velocity="1.0" />
+    <safety_controller k_velocity="10" k_position="15" soft_lower_limit="-0.05" soft_upper_limit="0.05" />
+    <origin xyz="${-(table_top_length)/3 + 0.15} 0.12 ${1e-1/3.2}" rpy="${0} 0 ${0}" />
+  </joint>
+  <joint name="table_to_leftneckbladder" type="fixed">
+    <parent link="table_top"/>
+    <child link="left_bladder"/>
+    <limit effort="200.0" lower="0.1016" upper="0.1016" velocity="1.0" />
+    <safety_controller k_velocity="10" k_position="15" soft_lower_limit="-0.05" soft_upper_limit="0.05" />
+    <origin xyz="${-(table_top_length)/3 + 0.15} -0.12 ${1e-1/3.2}" rpy="${0} 0 ${0}" />
+  </joint>
+  <!-- Actuator Links -->
+  <joint name="bigbladder_to_head" type="continuous">
+    <parent link="big_bladder_link"/>
+    <child link="headnball_link"/>
+    <limit effort="200.0" lower="0.1016" upper="0.1016" velocity="1.0" />
+    <safety_controller k_velocity="10" k_position="15" soft_lower_limit="-0.0" soft_upper_limit="0.3" />
+    <origin xyz="${(table_top_length)/5} 0 0" rpy="0 0 ${M_PI/2}" />
+  </joint>
+  <joint name="rightbladder_to_neck" type="continuous">
+    <parent link="right_bladder"/>
+    <child link="headnball_link"/>
+    <limit effort="200.0" lower="0.1016" upper="0.1016" velocity="1.0" />
+    <safety_controller k_velocity="10" k_position="15" soft_lower_limit="-0.0" soft_upper_limit="0.3" />
+    <origin xyz="0 0 0" rpy="0 0 ${M_PI/2}" />
+  </joint>
+  <joint name="leftbladder_to_neck" type="continuous">
+    <parent link="left_bladder"/>
+    <child link="headnball_link"/>
+    <limit effort="200.0" lower="0.1016" upper="0.1016" velocity="1.0" />
+    <safety_controller k_velocity="10" k_position="15" soft_lower_limit="0.0" soft_upper_limit="0.3" />
+    <origin xyz="0 0 0" rpy="0 0 ${M_PI/2}" />
+  </joint>
+  <joint name="tableTop_to_basePanel" type="fixed">
     <parent link="table_top"/>
     <child link="base_panel"/>
-    <origin xyz="${bladder_pos_x + .08} ${bladder_pos_y + .23} ${(panel_thickness/2)}" rpy="0 0 ${PI/2}" />
+    <origin xyz="${-(table_top_length)/2 + 0.15} 0 ${1e-1/8}" rpy="${0} 0 ${M_PI/2}" />
   </joint>
-   <joint name="bladder_to_headnball" type="continuous">
-    <parent link="bladder_link"/>
-    <child link="headnball_link"/>
-    <limit effort="200.0" lower="0.1016" upper="0.1016" velocity="1.0" />
-    <safety_controller k_velocity="10" k_position="15" soft_lower_limit="-0.01" soft_upper_limit="0.3" />
-    <origin xyz="0.3 ${bladder_pos_y+0.35} ${0.5}" rpy="${-M_PI/2} 0 0" />
-   </joint>
-  <!-- Motion capture to base link -->
-  <joint name="motion_capture_to_world" type="fixed">
+  <joint name="vicon_to_world" type="fixed">
     <parent link="world"/>
-    <child link="motion_capture_frame"/>
-    <origin xyz="-5 -4 2.54" rpy="0 0 0" />
+    <child link="vicon_frame"/>
+    <origin xyz="-5 -4 2.00" rpy="0 0 0" />
   </joint>
 </robot>

File: superchick/table.xacro (robot description, xacro)
@@ -64,4 +64,5 @@
       </geometry>
     </collision>
+    <!-- KDL does not support root link inertia mass -->
   </link>
 <!-- right leg -->
@@ -82,5 +83,5 @@
     <inertial>
       <origin xyz="0 0 0" rpy="0 0 0" />
-      <mass value="10"/>
+      <mass value="0.1"/>
       <inertia ixx="1e-1" ixy="0.0" ixz="0.0" iyy="1e-1" iyz="0.0" izz="1e-1"/>
     </inertial>
@@ -108,6 +109,7 @@
     </collision>
     <inertial>
-      <mass value="10"/>
-      <inertia ixx="1.0" ixy="0.0" ixz="0.0" iyy="1.0" iyz="0.0" izz="1.0"/>
+      <origin xyz="0 0 0" rpy="0 0 0" />
+      <mass value="0.1"/>
+      <inertia ixx="1e-1" ixy="0.0" ixz="0.0" iyy="1e-1" iyz="0.0" izz="1e-1"/>
     </inertial>
   </link>
@@ -134,6 +136,7 @@
     </collision>
     <inertial>
-      <mass value="10"/>
-       <inertia ixx="1.0" ixy="0.0" ixz="0.0" iyy="1.0" iyz="0.0" izz="1.0"/>
+      <origin xyz="0 0 0" rpy="0 0 0" />
+      <mass value="0.1"/>
+      <inertia ixx="1e-1" ixy="0.0" ixz="0.0" iyy="1e-1" iyz="0.0" izz="1e-1"/>
     </inertial>
   </link>
@@ -163,6 +166,7 @@
     </collision>
     <inertial>
-      <mass value="10"/>
-       <inertia ixx="1.0" ixy="0.0" ixz="0.0" iyy="1.0" iyz="0.0" izz="1.0"/>
+      <origin xyz="0 0 0" rpy="0 0 0" />
+      <mass value="1e-1"/>
+      <inertia ixx="1e-1" ixy="0.0" ixz="0.0" iyy="1e-1" iyz="0.0" izz="1e-1"/>
     </inertial>
   </link>
@@ -172,15 +176,3 @@
     <origin xyz="0 ${(table_top_width/2)-0.08} -0.18" rpy="${-M_PI/2} 0 0 "/>
   </joint>
-<!--
-  <joint name="left_leg_to_tablecover" type="fixed">
-    <parent link="table_top"/>
-    <child link="left_leg"/>
-    <origin xyz="0 ${(table_top_width/2)-0.08} -0.18" rpy="${-M_PI/2} 0 0 "/>
-  </joint>
-  <joint name="right_leg_to_tablecover" type="fixed">
-    <parent link="table_top"/>
-    <child link="right_leg"/>
-    <origin xyz="0 ${(table_top_width/2)-0.08} -0.18" rpy="${-M_PI/2} 0 0 "/>
-  </joint>
- -->
 </robot>

File: superchick/vicon.xacro (robot description, xacro)
@@ -2,29 +2,30 @@
 <robot name="vicon" xmlns:xacro="http://www.ros.org/wiki/xacro">
    <!-- General Properties -->
-   <xacro:property name="vicon_x" value="0.2794" />
-   <xacro:property name="z_from_table" value="4" />
-     <!-- Derived Variables -->
-  <material name="vicon_colors" >
-    <color rgba="0.133 0.55 0.13 1" /> <!--forest green-->
+    <!-- Constants -->
+  <xacro:property name="PI" value="3.14159" />
+  <material name="vicon_red" >
+    <color rgba="1 0 0 1" />
   </material>
-   <!-- inflatable air bladder -->
-   <link name="vicon_system">
-     <visual>
-       <origin xyz="0 0 0" rpy="0 0 0" />
-       <geometry>
-         <mesh filename="package://superchick/meshes/bladder.stl" scale=".001 .001 .001" />
-       </geometry>
-       <material name="bladder_color"/>
-       <origin xyz="0 0 0" rpy="0 0 0" />
-     </visual>
-     <collision>
-       <geometry>
-         <mesh filename="package://superchick/meshes/bladder.stl" scale=".001 .001 .001" />
-       </geometry>
-     </collision>
-     <inertial>
-       <mass value="10"/>
-       <inertia ixx="1.0" ixy="0.0" ixz="0.0" iyy="1.0" iyz="0.0" izz="1.0"/>
-     </inertial>
-   </link>
+  <!-- vicon Frame-->
+  <link name="vicon_frame">
+    <visual>
+      <origin xyz="0 0 0" rpy="${PI/2} 0 ${PI/2}" />
+      <geometry>
+        <mesh filename="package://superchick/meshes/vicon.stl" scale = ".001 .001 .001" />
+      </geometry>
+      <material name="vicon_red"/>
+    </visual>
+    <collision>
+      <origin xyz="0 0 0" rpy="${PI/2} 0 ${PI/2}" />
+      <geometry>
+        <mesh filename="package://superchick/meshes/vicon.stl" scale = ".001 .001 .001" />
+      </geometry>
+      <material name="vicon_red"/>
+    </collision>
+    <inertial>
+      <origin xyz="0 0 0" rpy="0 0 0" />
+      <mass value="1e-1"/>
+      <inertia ixx="1e-1" ixy="0.0" ixz="0.0" iyy="1e-1" iyz="0.0" izz="1e-1"/>
+    </inertial>
+  </link>
 </robot>
