Commit message: almost finished gazebo sim

File: superchick/cage.xacro (robot description, xacro)
@@ -60,5 +60,5 @@
 		<parent link="base_panel"/>
 		<child link="panel_12_oc"/>
-		<origin xyz="0 ${distance_panel_12_oc_from_center} ${(panel_thickness/2) + (panel_height/2)}" />
+		<origin xyz="0 ${1e-1} ${0.08/2.1}"/>
 	</joint>
 	<!-- 9:00 Panel -->

File: superchick/headnball.xacro (robot description, xacro)
@@ -12,11 +12,13 @@
    <link name="headnball_link">
      <visual>
-       <origin xyz="${0} ${head_y_orig} ${head_z_orig}" rpy="${M_PI/2} 0 ${-M_PI}" />
+       <origin xyz="${0} ${0} ${0}" rpy="${M_PI/2} 0 ${-M_PI}" />
        <geometry>
          <mesh filename="package://superchick/meshes/headnball.dae" scale=".001 .001 .001" />
        </geometry>
        <material name="brown"/>
-       <origin xyz="${0} ${head_y_orig} ${head_z_orig}" rpy="${M_PI/2} 0 ${-M_PI}" />
+       <origin xyz="${0} ${0} ${0}" rpy="${M_PI/2} 0 ${-M_PI}" />
      </visual>
+<!--
+After five days of trying, I realized that adding a collision object to a continuous link causes sdf to produce two separate joints
      <collision>
        <geometry>
@@ -25,15 +27,16 @@
        <origin xyz="${0} ${head_y_orig} ${head_z_orig}" rpy="${M_PI/2} 0 ${-M_PI}" />
      </collision>
-     <inertial>
+ -->
+<!--      <inertial>
        <mass value="${mass}"/>
        <inertia ixx="${mass/12}" ixy="0.0" ixz="0.0"
         iyy="${inertia_mom}" iyz="0.0000"
         izz="${inertia_mom}"/>
-     </inertial>
-<!--      <inertial>
+     </inertial> -->
+     <inertial>
        <mass value="1e-1"/>
        <inertia ixx="0.925288" ixy="0.379102" ixz="0.011081"
                 iyy="0.919140" iyz="0.111180" izz="0.993738"/>
-     </inertial> -->
+     </inertial>
    </link>
 </robot>

File: superchick/superchick.xacro (robot description, xacro)
@@ -12,5 +12,5 @@
    <xacro:include filename="$(find superchick)/bladders.xacro" />
    <xacro:include filename="$(find superchick)/headnball.xacro" />
-   <xacro:include filename="$(find superchick)/cage.xacro" />
+   <!-- <xacro:include filename="$(find superchick)/cage.xacro" /> -->
    <xacro:include filename="$(find superchick)/vicon.xacro" />
    <xacro:if value="${sim == 'true'}">
@@ -23,5 +23,5 @@
     <limit effort="200.0" lower="0.1016" upper="0.1016" velocity="1.0" />
     <safety_controller k_velocity="10" k_position="15" soft_lower_limit="-0.05" soft_upper_limit="0.05" />
-    <origin xyz="${-(table_top_length)/2 + 0.23} 0 ${1e-1/3}" rpy="${0} 0 ${0}" />
+    <origin xyz="${-(table_top_length)/6} 0 ${0}" rpy="${0} 0 ${0}" />
   </joint>
   <!-- Actuator Links -->
@@ -32,6 +32,6 @@
     <limit effort="200.0" lower="-0.1016" upper="0.1016" velocity="1.0" />
     <dynamics damping="${damping}" friction="${friction}" />
-    <safety_controller k_velocity="10" k_position="15" soft_lower_limit="-0.0" soft_upper_limit="0.3" />
-    <origin xyz="${(1e-1/2)+1e-1} ${(table_top_width)/6} 0" rpy="0 0 ${M_PI/2}" />
+    <safety_controller k_velocity="10" k_position="15" soft_lower_limit="0.0" soft_upper_limit="0.3" />
+    <origin xyz="${0.4} 0 ${0.1/6}" rpy="0 0 ${M_PI/2}" />
   </joint>
    <!-- Gazebo does not support parallel linkages -->
@@ -70,18 +70,12 @@
   </joint>
  -->
-  <joint name="tableTop_to_basePanel" type="fixed">
+<!--   <joint name="tableTop_to_basePanel" type="fixed">
     <parent link="table_top"/>
     <child link="base_panel"/>
-    <!-- <origin xyz="${-(table_top_length)/2 + 0.15} 0 ${1e-1/8}" rpy="${0} 0 ${M_PI/2}"  />-->
-     <origin xyz="${-(table_top_length)/2 + 0.15} 0 ${1e-1/8}" rpy="${0} 0 ${M_PI/2}"/>
-  </joint>
+     <origin xyz="${-(table_top_length)/2 + 0.15} 0 ${1e-1/8}" rpy="${0} 0 ${M_PI/2}"  />
+  </joint> -->
   <joint name="vicon_to_world" type="fixed">
     <parent link="world"/>
     <child link="vicon_frame"/>
-    <origin xyz="-3.5 -2.0 -0.2" rpy="0 0 0" />
-  </joint>
-  <joint name="table_to_world" type="fixed">
-    <parent link="world"/>
-    <child link="table_top"/>
     <origin xyz="-3.5 -2.0 -0.2" rpy="0 0 0" />
   </joint>

File: superchick/table.xacro (robot description, xacro)
@@ -45,5 +45,5 @@
     </collision>
     <inertial>
-      <mass value="1"/>
+      <mass value="0.1"/>
         <inertia ixx="0.13" iyy="0.524" izz="0.539" ixy="0" ixz="0" iyz="0" />
     </inertial>
@@ -131,5 +131,5 @@
     <parent link="right_leg"/>
     <child link="table_top" />
-    <origin xyz="${-(table_top_length/2)+0.0762} 0 0.35 " />
+    <origin xyz="-0.35 0 0.17 " />
   </joint>
   <joint name="leftleg_to_tabletop" type="fixed">
@@ -142,14 +142,14 @@
       <origin xyz="0 0 ${-table_top_thickness}" rpy="0 0 0" />
       <geometry>
-        <box size="${table_cover_length} ${table_cover_width} ${table_cover_thickness}" />
+        <box size="${table_cover_length} ${table_cover_width/2} ${table_cover_thickness}" />
       </geometry>
       <material name="table_cover_color"/>
       <origin xyz="0 0 ${-table_top_thickness}" rpy="0 0 0" />
     </visual>
-    <collision>
+<!--     <collision>
       <geometry>
-        <box size="${table_cover_length} ${table_cover_width} ${table_cover_thickness}" />
+        <box size="${table_cover_length} ${table_cover_width/2} ${table_cover_thickness}" />
       </geometry>
-    </collision>
+    </collision> -->
     <inertial>
       <mass value="${mass}"/>
@@ -162,5 +162,5 @@
     <parent link="table_top"/>
     <child link="table_cover"/>
-    <origin xyz="0 ${(table_top_width/2)-0.08} -0.18" rpy="${-M_PI/2} 0 0 "/>
+    <origin xyz="0 0 ${0.05/4}" rpy="${-M_PI/2} 0 0 "/>
   </joint>
 </robot>
