Commit message: edited srdf files

File: superchick/superchick.xacro (robot description, xacro)
@@ -10,5 +10,5 @@
    <xacro:include filename="$(find superchick)/headnball.xacro" ns="headnball_ns" />
    <!-- table link to bladder -->
-   <joint name="table_to_bladder" type="planar">
+   <joint name="table_to_bladder" type="fixed">
     <parent link="table_top"/>
     <child link="bladder_link"/>

File: superchick/table.xacro (robot description, xacro)
@@ -64,8 +64,8 @@
       </geometry>
     </collision>
-    <inertial>
+<!--     <inertial>
       <mass value="10"/>
       <inertia ixx="1.0" ixy="0.0" ixz="0.0" iyy="1.0" iyz="0.0" izz="1.0"/>
-    </inertial>
+    </inertial> -->
   </link>
 <!-- right leg -->
@@ -175,3 +175,15 @@
     <origin xyz="0 ${(table_top_width/2)-0.08} -0.18" rpy="${-M_PI/2} 0 0 "/>
   </joint>
+<!--
+  <joint name="left_leg_to_tablecover" type="fixed">
+    <parent link="table_top"/>
+    <child link="left_leg"/>
+    <origin xyz="0 ${(table_top_width/2)-0.08} -0.18" rpy="${-M_PI/2} 0 0 "/>
+  </joint>
+  <joint name="right_leg_to_tablecover" type="fixed">
+    <parent link="table_top"/>
+    <child link="right_leg"/>
+    <origin xyz="0 ${(table_top_width/2)-0.08} -0.18" rpy="${-M_PI/2} 0 0 "/>
+  </joint>
+ -->
 </robot>

Commit message: Alex's addition of the motion capture system

File: superchick/superchick.xacro (robot description, xacro)
@@ -10,4 +10,5 @@
    <xacro:include filename="$(find superchick)/headnball.xacro" ns="headnball_ns" />
    <xacro:include filename="$(find superchick)/cage.xacro" ns="cage_ns" />
+   <xacro:include filename="$(find superchick)/motionCaptureSystem.xacro" ns="motionCaptureSystem_ns" />
    <!-- table link to bladder -->
     <joint name="table_to_bladder" type="fixed">
@@ -40,4 +41,10 @@
     <origin xyz="0.3 ${bladder_pos_y+0.35} ${0.5}" rpy="${-M_PI/2} 0 0" />
    </joint>
+  <!-- Motion capture to base link -->
+  <joint name="motion_capture_to_base_link" type="fixed">
+    <parent link="base_link"/>
+    <child link="motion_capture_frame"/>
+    <origin xyz="-5 -4 2.54" rpy="0 0 0" />
+  </joint>
 </robot>
 <!-- ${(table_top_length/2)-0.6} -->

Commit message: gazebo model loads but joints displaced

File: superchick/superchick.xacro (robot description, xacro)
@@ -1,5 +1,4 @@
 <?xml version="1.0"?>
 <robot name="superchick" xmlns:xacro="http://www.ros.org/wiki/xacro">
-  <xacro:include filename="$(find superchick)/superchick.gazebo" />
    <!-- General Properties -->
    <xacro:property name="bladder_pos_x" value="-0.7" />
@@ -14,4 +13,5 @@
    <xacro:include filename="$(find superchick)/cage.xacro" />
    <xacro:include filename="$(find superchick)/vicon.xacro" />
+   <xacro:include filename="$(find superchick)/superchick.gazebo" />
    <!-- table link to bladders -->
   <joint name="table_to_big_bladder" type="fixed">

File: superchick/vicon.xacro (robot description, xacro)
@@ -1,10 +1,8 @@
 <?xml version="1.0"?>
 <robot name="superchick" xmlns:xacro="http://www.ros.org/wiki/xacro">
-   <!-- General Properties -->
-  <xacro:property name="PI" value="3.14159" />
   <!-- vicon Frame-->
   <link name="vicon_frame">
     <visual>
-      <origin xyz="0 0 0" rpy="${PI/2} 0 ${PI/2}" />
+      <origin xyz="0 0 0" rpy="${M_PI/2} 0 ${M_PI/2}" />
       <geometry>
         <mesh filename="package://superchick/meshes/vicon2.dae" scale = ".001 .001 .001" />
@@ -13,5 +11,5 @@
     </visual>
     <collision>
-      <origin xyz="0 0 0" rpy="${PI/2} 0 ${PI/2}" />
+      <origin xyz="0 0 0" rpy="${M_PI/2} 0 ${M_PI/2}" />
       <geometry>
         <mesh filename="package://superchick/meshes/vicon2.dae" scale = ".001 .001 .001" />

Commit message: added transmission to actuator joints

File: superchick/superchick.xacro (robot description, xacro)
@@ -6,4 +6,5 @@
    <xacro:property name="damping" value="0.1" />
    <xacro:property name="friction" value="0.2" />
+   <xacro:property name="sim" value="false" />
   <!-- This file contains the table and bladder descriptions -->
    <xacro:include filename="$(find superchick)/material.xacro" />
@@ -13,5 +14,7 @@
    <xacro:include filename="$(find superchick)/cage.xacro" />
    <xacro:include filename="$(find superchick)/vicon.xacro" />
-   <xacro:include filename="$(find superchick)/superchick.gazebo" />
+   <xacro:if value="${sim == 'true'}">
+    <xacro:include filename="$(find superchick)/superchick.gazebo" />
+   </xacro:if>
    <!-- table link to bladders -->
   <joint name="table_to_big_bladder" type="fixed">
@@ -72,5 +75,35 @@
     <parent link="world"/>
     <child link="vicon_frame"/>
-    <origin xyz="-5 -4 2.00" rpy="0 0 0" />
+    <origin xyz="-3.5 -2.0 -0.2" rpy="0 0 0" />
   </joint>
+  <transmission name="base_transmission">
+     <type>transmission_interface/SimpleTransmission</type>
+     <joint name="joint1">
+       <hardwareInterface>EffortJointInterface</hardwareInterface>
+     </joint>
+     <actuator name="base_bladder">
+       <hardwareInterface>EffortJointInterface</hardwareInterface>
+       <mechanicalReduction>1</mechanicalReduction>
+     </actuator>
+   </transmission>
+   <transmission name="right_transmission">
+      <type>transmission_interface/SimpleTransmission</type>
+      <joint name="rightbladder_to_neck">
+        <hardwareInterface>EffortJointInterface</hardwareInterface>
+      </joint>
+      <actuator name="right_bladder">
+        <hardwareInterface>EffortJointInterface</hardwareInterface>
+        <mechanicalReduction>1</mechanicalReduction>
+      </actuator>
+    </transmission>
+    <transmission name="left_transmission">
+       <type>transmission_interface/SimpleTransmission</type>
+       <joint name="leftbladder_to_neck">
+         <hardwareInterface>EffortJointInterface</hardwareInterface>
+       </joint>
+       <actuator name="left_bladder">
+         <hardwareInterface>EffortJointInterface</hardwareInterface>
+         <mechanicalReduction>1</mechanicalReduction>
+       </actuator>
+     </transmission>
 </robot>

File: superchick/table.xacro (robot description, xacro)
@@ -8,5 +8,5 @@
         roslaunch superchick display.launch model:=table.urdf
   -->
-  <xacro:property name="M_PI" value="3.14159" />
+  <xacro:property name="M_PI" value="${22/7}" />
   <!-- table top properties -->
   <xacro:property name="table_top_length" value="1.524" />

File: superchick/vicon.xacro (robot description, xacro)
@@ -6,5 +6,5 @@
       <origin xyz="0 0 0" rpy="${M_PI/2} 0 ${M_PI/2}" />
       <geometry>
-        <mesh filename="package://superchick/meshes/vicon2.dae" scale = ".001 .001 .001" />
+        <mesh filename="package://superchick/meshes/vicon3.dae" scale = ".001 .001 .001" />
       </geometry>
       <material name="vicon_red"/>
@@ -13,5 +13,5 @@
       <origin xyz="0 0 0" rpy="${M_PI/2} 0 ${M_PI/2}" />
       <geometry>
-        <mesh filename="package://superchick/meshes/vicon2.dae" scale = ".001 .001 .001" />
+        <mesh filename="package://superchick/meshes/vicon3.dae" scale = ".001 .001 .001" />
       </geometry>
       <material name="vicon_red"/>

Commit message: with right bladder joint only

File: superchick/superchick.xacro (robot description, xacro)
@@ -28,4 +28,5 @@
     <parent link="table_top"/>
     <child link="right_bladder"/>
+    <dynamics damping="0.1"/>
     <limit effort="200.0" lower="0.1016" upper="0.1016" velocity="1.0" />
     <safety_controller k_velocity="10" k_position="15" soft_lower_limit="-0.05" soft_upper_limit="0.05" />
