Commit message: added newly trained controller mlp

File: superchick/superchick.urdf (robot description, URDF)
Before this commit: robot superchick, 14 links, 16 joints
Links:
- link vicon_frame: geometry collision mesh filename=package://superchick/meshes/vicon3.dae scale=.001 .001 .001; visual mesh filename=package://superchick/meshes/vicon3.dae scale=.001 .001 .001
Joints:
- joint vicon_to_world: origin xyz=-5 -4 2.00 rpy=0 0 0 -> xyz=-3.5 -2.0 -0.2 rpy=0 0 0

Commit message: dont use kinematic chain or native ik solver; single-bladder iab for dp project

File: superchick/superchick.urdf (robot description, URDF)
Before this commit: robot superchick, 14 links, 16 joints
Links:
- removed link left_bladder
- removed link right_bladder
- link vicon_frame: geometry collision mesh filename=package://superchick/meshes/vicon3.dae scale=.001 .001 .001; visual mesh filename=package://superchick/meshes/vicon3.dae scale=.001 .001 .001
Joints:
- removed joint leftbladder_to_neck
- removed joint rightbladder_to_neck
- removed joint table_to_leftneckbladder
- removed joint table_to_rightneckbladder
- joint vicon_to_world: origin xyz=-5 -4 2.00 rpy=0 0 0 -> xyz=-3.5 -2.0 -0.2 rpy=0 0 0

File: superchick/superchick.xacro (robot description, xacro)
@@ -15,5 +15,5 @@
    <xacro:include filename="$(find superchick)/vicon.xacro" />
    <xacro:if value="${sim == 'true'}">
-    <xacro:include filename="$(find superchick)/superchick.gazebo" />
+    <xacro:include filename="$(find superchick_gazebo)/superchick.gazebo" />
    </xacro:if>
    <!-- table link to bladders -->
@@ -25,5 +25,5 @@
     <origin xyz="${-(table_top_length)/2 + 0.23} 0 ${1e-1/3}" rpy="${0} 0 ${0}" />
   </joint>
-  <joint name="table_to_rightneckbladder" type="fixed">
+<!--   <joint name="table_to_rightneckbladder" type="fixed">
     <parent link="table_top"/>
     <child link="right_bladder"/>
@@ -39,5 +39,5 @@
     <safety_controller k_velocity="10" k_position="15" soft_lower_limit="-0.05" soft_upper_limit="0.05" />
     <origin xyz="${-(table_top_length)/3 + 0.15} -0.12 ${1e-1/3.2}" rpy="${0} 0 ${0}" />
-  </joint>
+  </joint> -->
   <!-- Actuator Links -->
   <joint name="bigbladder_to_head" type="continuous">
@@ -46,11 +46,13 @@
     <child link="headnball_link"/>
     <limit effort="200.0" lower="-0.1016" upper="0.1016" velocity="1.0" />
-    <safety_controller k_velocity="10" k_position="15" soft_lower_limit="-0.0" soft_upper_limit="0.3" />
+    <dynamics damping="${damping}" friction="${friction}" />
+    <safety_controller k_velocity="10" k_position="15" soft_lower_limit="0.0" soft_upper_limit="${2*0.3}" />
     <origin xyz="${(1e-1/2)+1e-1} ${(table_top_width)/6} 0" rpy="0 0 ${M_PI/2}" />
   </joint>
-  <joint name="rightbladder_to_neck" type="continuous">
+<!--   <joint name="rightbladder_to_neck" type="continuous">
     <axis xyz="1 -1 0" rpy="0 0 0" />
-    <parent link="right_bladder"/>
-    <child link="headnball_link"/>
+    <mimic joint="bigbladder_to_head" multiplier="1" offset="0"/>
+    <parent link="headnball_link"/>
+    <child link="right_bladder"/>
     <limit effort="200.0" lower="-0.1016" upper="0.1016" velocity="1.0" />
     <dynamics damping="${damping}" friction="${friction}" />
@@ -60,4 +62,5 @@
   <joint name="leftbladder_to_neck" type="continuous">
     <axis xyz="1 1 0" rpy="0 0 0" />
+    <mimic joint="bigbladder_to_head" multiplier="1" offset="0"/>
     <parent link="left_bladder"/>
     <child link="headnball_link"/>
@@ -67,5 +70,5 @@
     <dynamics damping="${damping}" friction="${friction}" />
     <origin xyz="0 0.25 0" rpy="0 0 ${M_PI/2}" />
-  </joint>
+  </joint>  -->
   <joint name="tableTop_to_basePanel" type="fixed">
     <parent link="table_top"/>
@@ -80,5 +83,5 @@
   <transmission name="base_transmission">
      <type>transmission_interface/SimpleTransmission</type>
-     <joint name="joint1">
+     <joint name="bigbladder_to_head">
        <hardwareInterface>EffortJointInterface</hardwareInterface>
      </joint>
@@ -88,5 +91,5 @@
      </actuator>
    </transmission>
-   <transmission name="right_transmission">
+<!--    <transmission name="right_transmission">
       <type>transmission_interface/SimpleTransmission</type>
       <joint name="rightbladder_to_neck">
@@ -107,4 +110,4 @@
          <mechanicalReduction>1</mechanicalReduction>
        </actuator>
-     </transmission>
+     </transmission> -->
 </robot>
