Commit message: updated chick

File: superchick/bladders.xacro (robot description, xacro)
@@ -6,7 +6,7 @@
    <xacro:property name="bladder_width" value="0.15748" />
    <xacro:property name="bladder_thickness" value="0.0508" />
-   <!-- this is used in calculating the size of the big bladder
-   Should be 2 ideally but too lay to fix associated deps -->
-   <xacro:property name="bladder_constant" value="1.5" />
+   <xacro:property name="bladder_constant" value="2" />
+   <xacro:property name="left_bladder_x" value="${bladder_width/2}" />
+   <!-- <xacro:property name="left_bladder_y" value="${bladder_width/2}" /> -->
      <!-- Derived Variables -->
   <material name="bladder_color" >

File: superchick/headnball.xacro (robot description, xacro)
@@ -7,5 +7,5 @@
    <xacro:property name="M_PI" value="3.14159" ns="headnball"/>
   <xacro:property name="head_x_orig" value="-0.1" />
-  <xacro:property name="head_y_orig" value="0.25" />
+  <xacro:property name="head_y_orig" value="${1.5*-1e-1}" />
   <material name="brown">
   <color rgba="0.647059 0.164706 0.164706 1"/>
@@ -14,10 +14,10 @@
    <link name="headnball_link">
      <visual>
-       <origin xyz="${0} ${0} ${-0.05}" rpy="${M_PI/2} 0 ${-M_PI}" />
+       <origin xyz="${0} ${head_y_orig} ${0}" rpy="${M_PI/2} 0 ${-M_PI}" />
        <geometry>
          <mesh filename="package://superchick/meshes/headnball.dae" scale=".001 .001 .001" />
        </geometry>
        <material name="brown"/>
-       <origin xyz="${0} ${0} ${0}" rpy="${M_PI/2} 0 ${-M_PI}" />
+       <origin xyz="${0} ${head_y_orig} ${0}" rpy="${M_PI/2} 0 ${-M_PI}" />
      </visual>
      <collision>
@@ -25,5 +25,5 @@
          <mesh filename="package://superchick/meshes/headnball.dae" scale=".001 .001 .001" />
        </geometry>
-       <origin xyz="${0} ${0} ${0}" rpy="${M_PI/2} 0 ${-M_PI}" />
+       <origin xyz="${0} ${head_y_orig} ${0}" rpy="${M_PI/2} 0 ${-M_PI}" />
      </collision>
      <inertial>

File: superchick/superchick.xacro (robot description, xacro)
@@ -16,5 +16,5 @@
     <limit effort="200.0" lower="0.1016" upper="0.1016" velocity="1.0" />
     <safety_controller k_velocity="10" k_position="15" soft_lower_limit="-0.05" soft_upper_limit="0.05" />
-    <origin xyz="${-(table_top_length)/2 + 0.2} 0 ${1e-1/3}" rpy="${0} 0 ${0}" />
+    <origin xyz="${-(table_top_length)/2 + 0.25} 0 ${1e-1/3}" rpy="${0} 0 ${0}" />
   </joint>
   <joint name="table_to_rightneckbladder" type="fixed">
@@ -30,5 +30,5 @@
     <limit effort="200.0" lower="0.1016" upper="0.1016" velocity="1.0" />
     <safety_controller k_velocity="10" k_position="15" soft_lower_limit="-0.05" soft_upper_limit="0.05" />
-    <origin xyz="${-(table_top_length)/3 + 0.15} -0.12 ${1e-1/3.2}" rpy="${0} 0 ${0}" />
+    <origin xyz="${-(table_top_length)/3 + 0.15} -0.01 ${1e-1/3.2}" rpy="${0} 0 ${0}" />
   </joint>
   <!-- Actuator Links -->
