Commit message: added axis to continuous joints

File: superchick/bladders.xacro (robot description, xacro)
@@ -1,17 +1,13 @@
 <?xml version="1.0"?>
-<robot name="bladder" xmlns:xacro="http://www.ros.org/wiki/xacro">
+<robot name="superchick" xmlns:xacro="http://www.ros.org/wiki/xacro">
    <!-- General Properties -->
    <!-- Lekan Ogunmolu | November 2016 -->
    <xacro:property name="bladder_length" value="0.15748" />
-   <xacro:property name="bladder_width" value="0.15748" />
+   <xacro:property name="bladder_width" value="${bladder_length}" />
    <xacro:property name="bladder_thickness" value="0.0508" />
    <xacro:property name="bladder_constant" value="2" />
    <xacro:property name="left_bladder_x" value="${bladder_width/2}" />
-   <!-- <xacro:property name="left_bladder_y" value="${bladder_width/2}" /> -->
-     <!-- Derived Variables -->
-  <material name="bladder_color" >
-    <color rgba="${255/255} ${255/255} 0 ${255/255}" />
-  </material>
-   <!-- inflatable air bladder -->
+   <xacro:property name="mass" value="1e-2" />
+   <xacro:property name="inertia_mom" value="${mass/12}" />
    <link name="right_bladder">
      <visual>
@@ -30,7 +26,8 @@
      </collision>
      <inertial>
-       <mass value="1e-2"/>
-       <inertia ixx="0.999998" ixy="0.0" ixz="0.0"
-        iyy="1.000000" iyz="-0.000011" izz="0.999998"/>
+       <mass value="${mass}"/>
+       <inertia ixx="${mass/12}" ixy="0.0" ixz="0.0"
+        iyy="${inertia_mom}" iyz="0.0000"
+        izz="${inertia_mom}"/>
      </inertial>
    </link>
@@ -51,7 +48,8 @@
      </collision>
      <inertial>
-       <mass value="1e-2"/>
-       <inertia ixx="0.999998" ixy="0.0" ixz="0.0"
-        iyy="1.000000" iyz="-0.000011" izz="0.999998"/>
+       <mass value="${mass}"/>
+       <inertia ixx="${mass/12}" ixy="0.0" ixz="0.0"
+        iyy="${inertia_mom}" iyz="0.0000"
+        izz="${inertia_mom}"/>
      </inertial>
    </link>
@@ -72,7 +70,8 @@
      </collision>
      <inertial>
-       <mass value="1e-2"/>
-       <inertia ixx="0.999998" ixy="0.0" ixz="0.0"
-        iyy="1.000000" iyz="-0.000011" izz="0.999998"/>
+       <mass value="${mass}"/>
+       <inertia ixx="${mass/12}" ixy="0.0" ixz="0.0"
+        iyy="${inertia_mom}" iyz="0.0000"
+        izz="${inertia_mom}"/>
      </inertial>
    </link>

File: superchick/cage.xacro (robot description, xacro)
@@ -1,13 +1,11 @@
 <?xml version="1.0"?>
-<robot name="cage" xmlns:xacro="http://www.ros.org/wiki/xacro">
+<robot name="superchick" xmlns:xacro="http://www.ros.org/wiki/xacro">
 	<!-- Description: Head Cage
 	 Author: Alex Tomkovich, September 27, 2016
 	 Modified: Lekan Ogunmolu Nov. 18, 2016
  	-->
-	<!-- Constants -->
-	<xacro:property name="PI" value="3.14159" />
 	<!-- Panel Properties -->
 	<xacro:property name="side_panel_length" value=".231775" />
-	<xacro:property name="panel_12_oc_length" value=".4700" /> <!--.34925 -->
+	<xacro:property name="panel_12_oc_length" value=".4700" />
 	<xacro:property name="panel_height" value=".200025" />
 	<xacro:property name="panel_thickness" value=".0047625" />
@@ -15,9 +13,4 @@
 	<xacro:property name="base_panel_width" value=".2794" />
 	<xacro:property name ="distance_panel_12_oc_from_center" value ="${(base_panel_width/2) - .04572}" />
-	<!-- Derived Variables -->
-	<material name="panel_color" >
-		<color rgba="0.133 0.55 0.13 1" />
-	</material>
-	<!-- Base panel -->
 	<link name="base_panel">
 		<visual>
@@ -35,7 +28,8 @@
 		</collision>
 		<inertial>
-		  <origin xyz="0 0 0" rpy="0 0 0" />
-		  <mass value="0.1"/>
-		  <inertia ixx="1e-1" ixy="0.0" ixz="0.0" iyy="1e-1" iyz="0.0" izz="1e-1"/>
+		  <mass value="${mass}"/>
+		  <inertia ixx="${mass/12}" ixy="0.0" ixz="0.0"
+		   iyy="${inertia_mom}" iyz="0.0000"
+		   izz="${inertia_mom}"/>
 		</inertial>
 	</link>
@@ -47,5 +41,5 @@
 			</geometry>
 			<material name="panel_color" />
-			<origin xyz="0 0 0" rpy="${(PI/2)} 0 0" />
+			<origin xyz="0 0 0" rpy="${(M_PI/2)} 0 0" />
 		</visual>
 		<collision>
@@ -53,14 +47,15 @@
 				<box size="${panel_12_oc_length} ${panel_height} ${panel_thickness}" />
 			</geometry>
-			<origin xyz="0 0 0" rpy="${(PI/2)} 0 0" />
+			<origin xyz="0 0 0" rpy="${(M_PI/2)} 0 0" />
 		</collision>
 		<inertial>
-		  <origin xyz="0 0 0" rpy="0 0 0" />
-		  <mass value="0.1"/>
-		  <inertia ixx="1e-1" ixy="0.0" ixz="0.0" iyy="1e-1" iyz="0.0" izz="1e-1"/>
+		  <mass value="${mass}"/>
+		  <inertia ixx="${mass/12}" ixy="0.0" ixz="0.0"
+		   iyy="${inertia_mom}" iyz="0.0000"
+		   izz="${inertia_mom}"/>
 		</inertial>
 	</link>
 	<!-- Join 12:00 Panel to base_panel -->
-	<joint name="panel_12_oc_to_base_panel" type="fixed">
+	<joint name="base_panel_to_12oc" type="fixed">
 		<parent link="base_panel"/>
 		<child link="panel_12_oc"/>
@@ -70,5 +65,5 @@
 	<link name="panel_9_oc">
 		<visual>
-			<origin xyz="0 0 0" rpy="${(PI/2)} 0 ${(PI/2)}" />
+			<origin xyz="0 0 0" rpy="${(M_PI/2)} 0 ${(M_PI/2)}" />
 			<geometry>
 				<box size="${side_panel_length} ${panel_height} ${panel_thickness}" />
@@ -80,14 +75,15 @@
 				<box size="${side_panel_length} ${panel_height} ${panel_thickness}" />
 			</geometry>
-			<origin xyz="0 0 0" rpy="${(PI/2)} 0 ${(PI/2)}" />
+			<origin xyz="0 0 0" rpy="${(M_PI/2)} 0 ${(M_PI/2)}" />
 		</collision>
 		<inertial>
-		  <origin xyz="0 0 0" rpy="0 0 0" />
-		  <mass value="0.1"/>
-		  <inertia ixx="1e-1" ixy="0.0" ixz="0.0" iyy="1e-1" iyz="0.0" izz="1e-1"/>
+		  <mass value="${mass}"/>
+		  <inertia ixx="${mass/12}" ixy="0.0" ixz="0.0"
+		   iyy="${inertia_mom}" iyz="0.0000"
+		   izz="${inertia_mom}"/>
 		</inertial>
 	</link>
 	<!-- Join 9:00 Panel to 12:00 Panel -->
-	<joint name="panel_9_oc_to_panel_12_oc" type="fixed">
+	<joint name="12oc_to_9oc" type="fixed">
 		<parent link="panel_12_oc"/>
 		<child link="panel_9_oc"/>
@@ -97,5 +93,5 @@
 	<link name="panel_3_oc">
 		<visual>
-			<origin xyz="0 0 0" rpy="${(PI/2)} 0 ${(PI/2)}" />
+			<origin xyz="0 0 0" rpy="${(M_PI/2)} 0 ${(M_PI/2)}" />
 			<geometry>
 				<box size="${side_panel_length} ${panel_height} ${panel_thickness}" />
@@ -107,14 +103,15 @@
 				<box size="${side_panel_length} ${panel_height} ${panel_thickness}" />
 			</geometry>
-			<origin xyz="0 0 0" rpy="${(PI/2)} 0 ${(PI/2)}" />
+			<origin xyz="0 0 0" rpy="${(M_PI/2)} 0 ${(M_PI/2)}" />
 		</collision>
 		<inertial>
-		  <origin xyz="0 0 0" rpy="0 0 0" />
-		  <mass value="0.1"/>
-		  <inertia ixx="1e-1" ixy="0.0" ixz="0.0" iyy="1e-1" iyz="0.0" izz="1e-1"/>
+		  <mass value="${mass}"/>
+		  <inertia ixx="${mass/12}" ixy="0.0" ixz="0.0"
+		   iyy="${inertia_mom}" iyz="0.0000"
+		   izz="${inertia_mom}"/>
 		</inertial>
 	</link>
 	<!-- Join 3:00 Panel to 12:00 Panel -->
-	<joint name="panel_3_oc_to_panel_12_oc" type="fixed">
+	<joint name="12oc_to_3oc" type="fixed">
 		<parent link="panel_12_oc"/>
 		<child link="panel_3_oc"/>

File: superchick/headnball.xacro (robot description, xacro)
@@ -1,4 +1,4 @@
 <?xml version="1.0"?>
-<robot name="white_head" xmlns:xacro="http://www.ros.org/wiki/xacro">
+<robot name="superchick" xmlns:xacro="http://www.ros.org/wiki/xacro">
    <!-- General Properties -->
    <xacro:property name="head_height" value="0.2794" />
@@ -6,30 +6,34 @@
    <xacro:property name="head_thickness" value="0.1778" />
    <xacro:property name="M_PI" value="3.14159" ns="headnball"/>
-  <xacro:property name="head_x_orig" value="-0.1" />
-  <xacro:property name="head_y_orig" value="${1.5*-1e-1}" />
-  <material name="brown">
-  <color rgba="0.647059 0.164706 0.164706 1"/>
-  </material>
+   <xacro:property name="head_x_orig" value="-0.1" />
+   <xacro:property name="head_y_orig" value="${1.5*-1e-1}" />
+   <xacro:property name="head_z_orig" value="${0.11/3}" />
    <!-- inflatable air bladder -->
    <link name="headnball_link">
      <visual>
-       <origin xyz="${0} ${head_y_orig} ${0}" rpy="${M_PI/2} 0 ${-M_PI}" />
+       <origin xyz="${0} ${head_y_orig} ${head_z_orig}" rpy="${M_PI/2} 0 ${-M_PI}" />
        <geometry>
-         <mesh filename="package://superchick/meshes/headnball.dae" scale=".001 .001 .001" />
+         <mesh filename="package://superchick/meshes/headnball.stl" scale=".001 .001 .001" />
        </geometry>
        <material name="brown"/>
-       <origin xyz="${0} ${head_y_orig} ${0}" rpy="${M_PI/2} 0 ${-M_PI}" />
+       <origin xyz="${0} ${head_y_orig} ${head_z_orig}" rpy="${M_PI/2} 0 ${-M_PI}" />
      </visual>
      <collision>
        <geometry>
-         <mesh filename="package://superchick/meshes/headnball.dae" scale=".001 .001 .001" />
+         <mesh filename="package://superchick/meshes/headnball.stl" scale=".001 .001 .001" />
        </geometry>
-       <origin xyz="${0} ${head_y_orig} ${0}" rpy="${M_PI/2} 0 ${-M_PI}" />
+       <origin xyz="${0} ${head_y_orig} ${head_z_orig}" rpy="${M_PI/2} 0 ${-M_PI}" />
      </collision>
      <inertial>
+       <mass value="${mass}"/>
+       <inertia ixx="${mass/12}" ixy="0.0" ixz="0.0"
+        iyy="${inertia_mom}" iyz="0.0000"
+        izz="${inertia_mom}"/>
+     </inertial>
+<!--      <inertial>
        <mass value="1e-1"/>
        <inertia ixx="0.925288" ixy="0.379102" ixz="0.011081"
                 iyy="0.919140" iyz="0.111180" izz="0.993738"/>
-     </inertial>
+     </inertial> -->
    </link>
 </robot>

File: superchick/novalis.xacro (robot description, xacro)
@@ -1,10 +1,6 @@
 <?xml version="1.0"?>
 <robot name="novalis" xmlns:xacro="http://www.ros.org/wiki/xacro">
-  <!-- Model for the Novalis Tx Spec
+  <!-- Part of the Model for the Novalis TX Spec
       Author: Olalekan Ogunmolu, August 2016
-        Generate urdf with
-        rosrun xacro xacro src/superchick/novalis.xacro > novalis.urdf
-        Then run with
-        roslaunch superchick display.launch model:=novalis.urdf
   -->
   <!-- General Properties -->

File: superchick/superchick.urdf (robot description, URDF)
Before this commit: robot superchick, 12 links, 12 joints
Links:
- removed link base_link
- removed link bladder_link
- removed link motion_capture_frame
- added link big_bladder_link, mass 0.01; collision box size=0.31496 0.31496 0.1016; visual box size=0.31496 0.31496 0.0508
- added link left_bladder, mass 0.01; collision box size=0.15748 0.15748 0.0508; visual box size=0.15748 0.15748 0.0508
- added link right_bladder, mass 0.01; collision box size=0.15748 0.15748 0.0508; visual box size=0.15748 0.15748 0.0508
- added link vicon_frame, mass 0.01; collision mesh filename=package://superchick/meshes/vicon2.dae scale=.001 .001 .001; visual mesh filename=package://superchick/meshes/vicon2.dae scale=.001 .001 .001
- added link world; collision box size=1.524 0.6198 0.0381; visual box size=1.524 0.6198 0.0381
- link base_panel: mass None -> 0.01
- link headnball_link: mass 10 -> 0.01; geometry collision mesh filename=package://superchick/meshes/headnball.dae scale=.001 .001 .001; visual mesh filename=package://superchick/meshes/headnball.dae scale=.001 .001 .001
- link left_leg: mass 10 -> 0.01
- link panel_12_oc: mass None -> 0.01
- link panel_3_oc: mass None -> 0.01
- link panel_9_oc: mass None -> 0.01
- link right_leg: mass 10 -> 0.01
- link table_cover: mass 10 -> 0.01
- link table_top: mass 10 -> 0.01
Joints:
- removed joint base_panel_to_table_top
- removed joint bladder_to_headnball
- removed joint motion_capture_to_base_link
- removed joint panel_12_oc_to_base_panel
- removed joint panel_3_oc_to_panel_12_oc
- removed joint panel_9_oc_to_panel_12_oc
- removed joint table_to_bladder
- added joint 12oc_to_3oc: type fixed, parent panel_12_oc, child panel_3_oc, origin xyz=0.23738125 -0.11350625 0
- added joint 12oc_to_9oc: type fixed, parent panel_12_oc, child panel_9_oc, origin xyz=-0.23738125 -0.11350625 0
- added joint base_panel_to_12oc: type fixed, parent base_panel, child panel_12_oc, origin xyz=0 0.09398 0.10239375
- added joint bigbladder_to_head: type continuous, parent big_bladder_link, child headnball_link, origin xyz=0.3048 0 0 rpy=0 0 1.570795, limit lower=0.1016 upper=0.1016 effort=200.0 velocity=1.0
- added joint leftbladder_to_neck: type continuous, parent left_bladder, child headnball_link, origin xyz=0 0 0 rpy=0 0 1.570795, limit lower=0.1016 upper=0.1016 effort=200.0 velocity=1.0
- added joint rightbladder_to_neck: type continuous, parent right_bladder, child headnball_link, origin xyz=0 0 0 rpy=0 0 1.570795, limit lower=0.1016 upper=0.1016 effort=200.0 velocity=1.0
- added joint tableTop_to_basePanel: type fixed, parent table_top, child base_panel, origin xyz=-0.612 0 0.0125 rpy=0.0 0 1.570795
- added joint table_to_big_bladder: type fixed, parent table_top, child big_bladder_link, origin xyz=-0.532 0 0.0333333333333 rpy=0.0 0 0.0, limit lower=0.1016 upper=0.1016 effort=200.0 velocity=1.0
- added joint table_to_leftneckbladder: type fixed, parent table_top, child left_bladder, origin xyz=-0.358 -0.12 0.03125 rpy=0.0 0 0.0, limit lower=0.1016 upper=0.1016 effort=200.0 velocity=1.0
- added joint table_to_rightneckbladder: type fixed, parent table_top, child right_bladder, origin xyz=-0.358 0.12 0.03125 rpy=0.0 0 0.0, limit lower=0.1016 upper=0.1016 effort=200.0 velocity=1.0
- added joint vicon_to_world: type fixed, parent world, child vicon_frame, origin xyz=-5 -4 2.00 rpy=0 0 0
- joint base_to_left_leg: parent base_link -> world
- joint base_to_right_leg: parent base_link -> world

File: superchick/superchick.xacro (robot description, xacro)
@@ -1,13 +1,15 @@
 <?xml version="1.0"?>
 <robot name="superchick" xmlns:xacro="http://www.ros.org/wiki/xacro">
+  <xacro:include filename="$(find superchick)/superchick.gazebo" />
    <!-- General Properties -->
    <xacro:property name="bladder_pos_x" value="-0.7" />
    <xacro:property name="bladder_pos_y" value="-0.35" />
   <!-- This file contains the table and bladder descriptions -->
-   <xacro:include filename="$(find superchick)/table.xacro" ns="table_ns" />
-   <xacro:include filename="$(find superchick)/bladders.xacro" ns="bladder_ns" />
-   <xacro:include filename="$(find superchick)/headnball.xacro" ns="headnball_ns" />
-   <xacro:include filename="$(find superchick)/cage.xacro" ns="cage_ns" />
-   <xacro:include filename="$(find superchick)/vicon.xacro" ns="vicon_ns" />
+   <xacro:include filename="$(find superchick)/material.xacro" />
+   <xacro:include filename="$(find superchick)/table.xacro" />
+   <xacro:include filename="$(find superchick)/bladders.xacro" />
+   <xacro:include filename="$(find superchick)/headnball.xacro" />
+   <xacro:include filename="$(find superchick)/cage.xacro" />
+   <xacro:include filename="$(find superchick)/vicon.xacro" />
    <!-- table link to bladders -->
   <joint name="table_to_big_bladder" type="fixed">
@@ -16,5 +18,5 @@
     <limit effort="200.0" lower="0.1016" upper="0.1016" velocity="1.0" />
     <safety_controller k_velocity="10" k_position="15" soft_lower_limit="-0.05" soft_upper_limit="0.05" />
-    <origin xyz="${-(table_top_length)/2 + 0.25} 0 ${1e-1/3}" rpy="${0} 0 ${0}" />
+    <origin xyz="${-(table_top_length)/2 + 0.23} 0 ${1e-1/3}" rpy="${0} 0 ${0}" />
   </joint>
   <joint name="table_to_rightneckbladder" type="fixed">
@@ -30,22 +32,25 @@
     <limit effort="200.0" lower="0.1016" upper="0.1016" velocity="1.0" />
     <safety_controller k_velocity="10" k_position="15" soft_lower_limit="-0.05" soft_upper_limit="0.05" />
-    <origin xyz="${-(table_top_length)/3 + 0.15} -0.01 ${1e-1/3.2}" rpy="${0} 0 ${0}" />
+    <origin xyz="${-(table_top_length)/3 + 0.15} -0.12 ${1e-1/3.2}" rpy="${0} 0 ${0}" />
   </joint>
   <!-- Actuator Links -->
   <joint name="bigbladder_to_head" type="continuous">
+    <axis xyz="1 0 0" rpy="0 0 0" />
     <parent link="big_bladder_link"/>
     <child link="headnball_link"/>
     <limit effort="200.0" lower="0.1016" upper="0.1016" velocity="1.0" />
     <safety_controller k_velocity="10" k_position="15" soft_lower_limit="-0.0" soft_upper_limit="0.3" />
-    <origin xyz="${(table_top_length)/5} 0 0" rpy="0 0 ${M_PI/2}" />
+    <origin xyz="${(table_top_length)/4} 0 0" rpy="0 0 ${M_PI/2}" />
   </joint>
   <joint name="rightbladder_to_neck" type="continuous">
+    <axis xyz="0 1 0" rpy="0 0 0" />
     <parent link="right_bladder"/>
     <child link="headnball_link"/>
-    <limit effort="200.0" lower="0.1016" upper="0.1016" velocity="1.0" />
-    <safety_controller k_velocity="10" k_position="15" soft_lower_limit="-0.0" soft_upper_limit="0.3" />
+    <limit effort="200.0" lower="0" upper="0.1016" velocity="1.0" />
+    <safety_controller k_velocity="10" k_position="15" soft_lower_limit="0.0" soft_upper_limit="-0.3" />
     <origin xyz="0 0 0" rpy="0 0 ${M_PI/2}" />
   </joint>
   <joint name="leftbladder_to_neck" type="continuous">
+    <axis xyz="0 0 1" rpy="0 0 0" />
     <parent link="left_bladder"/>
     <child link="headnball_link"/>

File: superchick/table.xacro (robot description, xacro)
@@ -1,4 +1,4 @@
 <?xml version="1.0"?>
-<robot name="acc16model" xmlns:xacro="http://www.ros.org/wiki/xacro">
+<robot name="superchick" xmlns:xacro="http://www.ros.org/wiki/xacro">
   <!-- Model for the Superchick Table Spec
       Author: Olalekan Ogunmolu, August 2016
@@ -8,5 +8,4 @@
         roslaunch superchick display.launch model:=table.urdf
   -->
-  <!-- General Properties -->
   <xacro:property name="M_PI" value="3.14159" />
   <!-- table top properties -->
@@ -30,23 +29,4 @@
   <xacro:property name="table_cover_width" value="0.2794" />
   <xacro:property name="table_cover_thickness" value="${0.127+0.1}" />
-  <!-- Derived Variables -->
-  <material name="table_color" >
-    <color rgba="0.8 0.8 0.8 1" />
-  </material>
-  <material name="blue">
-    <color rgba="0 0 .8 1"/>
-  </material>
-  <material name="table_cover_color">
-    <color rgba="0 ${26/255} ${51/255} 1"/>
-  </material>
-  <material name="dark_gray">
-    <color rgba="0.156863 0.156863 0.156863 1"/>
-  </material>
-  <material name="white">
-    <color rgba="1 1 1 1"/>
-  </material>
-  <material name="base_color">
-    <color rgba="0 0 0 0"/>
-  </material>
   <!-- table legs artificial base link -->
   <link name="world">
@@ -66,5 +46,5 @@
     <!-- KDL does not support root link inertia mass -->
   </link>
-<!-- right leg -->
+  <!-- right leg -->
   <link name="right_leg">
     <visual>
@@ -82,7 +62,8 @@
     </collision>
     <inertial>
-      <origin xyz="0 0 0" rpy="0 0 0" />
-      <mass value="0.1"/>
-      <inertia ixx="1e-1" ixy="0.0" ixz="0.0" iyy="1e-1" iyz="0.0" izz="1e-1"/>
+      <mass value="${mass}"/>
+      <inertia ixx="${mass/12}" ixy="0.0" ixz="0.0"
+       iyy="${inertia_mom}" iyz="0.0000"
+       izz="${inertia_mom}"/>
     </inertial>
   </link>
@@ -93,5 +74,5 @@
     <origin xyz="${(table_top_length/2)-0.0762} 0 0.3"/>
   </joint>
-<!-- draw left leg -->
+  <!-- draw left leg -->
   <link name="left_leg">
     <visual>
@@ -109,7 +90,8 @@
     </collision>
     <inertial>
-      <origin xyz="0 0 0" rpy="0 0 0" />
-      <mass value="0.1"/>
-      <inertia ixx="1e-1" ixy="0.0" ixz="0.0" iyy="1e-1" iyz="0.0" izz="1e-1"/>
+      <mass value="${mass}"/>
+      <inertia ixx="${mass/12}" ixy="0.0" ixz="0.0"
+        iyy="${inertia_mom}" iyz="0.0000"
+        izz="${inertia_mom}"/>
     </inertial>
   </link>
@@ -136,8 +118,9 @@
     </collision>
     <inertial>
-      <origin xyz="0 0 0" rpy="0 0 0" />
-      <mass value="0.1"/>
-      <inertia ixx="1e-1" ixy="0.0" ixz="0.0" iyy="1e-1" iyz="0.0" izz="1e-1"/>
-    </inertial>
+      <mass value="${mass}"/>
+      <inertia ixx="${mass/12}" ixy="0.0" ixz="0.0"
+        iyy="${inertia_mom}" iyz="0.0000"
+        izz="${inertia_mom}"/>
+      </inertial>
   </link>
   <joint name="rightleg_to_tabletop" type="fixed">
@@ -166,7 +149,8 @@
     </collision>
     <inertial>
-      <origin xyz="0 0 0" rpy="0 0 0" />
-      <mass value="1e-1"/>
-      <inertia ixx="1e-1" ixy="0.0" ixz="0.0" iyy="1e-1" iyz="0.0" izz="1e-1"/>
+      <mass value="${mass}"/>
+      <inertia ixx="${mass/12}" ixy="0.0" ixz="0.0"
+       iyy="${inertia_mom}" iyz="0.0000"
+       izz="${inertia_mom}"/>
     </inertial>
   </link>

File: superchick/vicon.xacro (robot description, xacro)
@@ -1,10 +1,6 @@
 <?xml version="1.0"?>
-<robot name="vicon" xmlns:xacro="http://www.ros.org/wiki/xacro">
+<robot name="superchick" xmlns:xacro="http://www.ros.org/wiki/xacro">
    <!-- General Properties -->
-    <!-- Constants -->
   <xacro:property name="PI" value="3.14159" />
-  <material name="vicon_red" >
-    <color rgba="1 0 0 1" />
-  </material>
   <!-- vicon Frame-->
   <link name="vicon_frame">
@@ -12,5 +8,5 @@
       <origin xyz="0 0 0" rpy="${PI/2} 0 ${PI/2}" />
       <geometry>
-        <mesh filename="package://superchick/meshes/vicon.stl" scale = ".001 .001 .001" />
+        <mesh filename="package://superchick/meshes/vicon2.dae" scale = ".001 .001 .001" />
       </geometry>
       <material name="vicon_red"/>
@@ -19,12 +15,13 @@
       <origin xyz="0 0 0" rpy="${PI/2} 0 ${PI/2}" />
       <geometry>
-        <mesh filename="package://superchick/meshes/vicon.stl" scale = ".001 .001 .001" />
+        <mesh filename="package://superchick/meshes/vicon2.dae" scale = ".001 .001 .001" />
       </geometry>
       <material name="vicon_red"/>
     </collision>
     <inertial>
-      <origin xyz="0 0 0" rpy="0 0 0" />
-      <mass value="1e-1"/>
-      <inertia ixx="1e-1" ixy="0.0" ixz="0.0" iyy="1e-1" iyz="0.0" izz="1e-1"/>
+      <mass value="${mass}"/>
+      <inertia ixx="${mass/12}" ixy="0.0" ixz="0.0"
+       iyy="${inertia_mom}" iyz="0.0000"
+       izz="${inertia_mom}"/>
     </inertial>
   </link>
