Commit message: updated all actuators

File: superchick/bladders.xacro (robot description, xacro)
@@ -34,10 +34,10 @@
    <link name="left_bladder">
      <visual>
-       <origin xyz="0 0 0" rpy="0 0 0" />
+       <origin xyz="0 ${0.1/2} 0" rpy="0 0 0" />
        <geometry>
          <box size="${bladder_length} ${bladder_width} ${bladder_thickness}" />
        </geometry>
        <material name="bladder_color"/>
-       <origin xyz="0 0 0" rpy="0 0 0" />
+       <origin xyz="0 ${0.1/2} 0" rpy="0 0 0" />
      </visual>
      <collision>
@@ -45,5 +45,5 @@
         <box size="${bladder_length} ${bladder_width} ${bladder_thickness}" />
        </geometry>
-       <origin xyz="0 0 0" rpy="0 0 0" />
+       <origin xyz="0 ${0.1/2} 0" rpy="0 0 0" />
      </collision>
      <inertial>

File: superchick/superchick.xacro (robot description, xacro)
@@ -5,4 +5,6 @@
    <xacro:property name="bladder_pos_x" value="-0.7" />
    <xacro:property name="bladder_pos_y" value="-0.35" />
+   <xacro:property name="damping" value="0.1" />
+   <xacro:property name="friction" value="0.2" />
   <!-- This file contains the table and bladder descriptions -->
    <xacro:include filename="$(find superchick)/material.xacro" />
@@ -39,23 +41,26 @@
     <parent link="big_bladder_link"/>
     <child link="headnball_link"/>
-    <limit effort="200.0" lower="0.1016" upper="0.1016" velocity="1.0" />
+    <limit effort="200.0" lower="-0.1016" upper="0.1016" velocity="1.0" />
     <safety_controller k_velocity="10" k_position="15" soft_lower_limit="-0.0" soft_upper_limit="0.3" />
-    <origin xyz="${(table_top_length)/4} 0 0" rpy="0 0 ${M_PI/2}" />
+    <origin xyz="${(1e-1/2)+1e-1} ${(table_top_width)/6} 0" rpy="0 0 ${M_PI/2}" />
   </joint>
   <joint name="rightbladder_to_neck" type="continuous">
-    <axis xyz="0 1 0" rpy="0 0 0" />
+    <axis xyz="1 -1 0" rpy="0 0 0" />
     <parent link="right_bladder"/>
     <child link="headnball_link"/>
-    <limit effort="200.0" lower="0" upper="0.1016" velocity="1.0" />
-    <safety_controller k_velocity="10" k_position="15" soft_lower_limit="0.0" soft_upper_limit="-0.3" />
+    <limit effort="200.0" lower="-0.1016" upper="0.1016" velocity="1.0" />
+    <dynamics damping="${damping}" friction="${friction}" />
+    <safety_controller k_velocity="10" k_position="15" soft_lower_limit="0.0" soft_upper_limit="0.3"/>
     <origin xyz="0 0 0" rpy="0 0 ${M_PI/2}" />
   </joint>
   <joint name="leftbladder_to_neck" type="continuous">
-    <axis xyz="0 0 1" rpy="0 0 0" />
+    <axis xyz="1 1 0" rpy="0 0 0" />
     <parent link="left_bladder"/>
     <child link="headnball_link"/>
-    <limit effort="200.0" lower="0.1016" upper="0.1016" velocity="1.0" />
+    <limit effort="200.0" lower="-0.1016" upper="0.1016" velocity="1.0" />
+    <dynamics damping="${damping}" friction="${friction}" />
     <safety_controller k_velocity="10" k_position="15" soft_lower_limit="0.0" soft_upper_limit="0.3" />
-    <origin xyz="0 0 0" rpy="0 0 ${M_PI/2}" />
+    <dynamics damping="${damping}" friction="${friction}" />
+    <origin xyz="0 0.25 0" rpy="0 0 ${M_PI/2}" />
   </joint>
   <joint name="tableTop_to_basePanel" type="fixed">

Commit message: creating gazebo branch

File: superchick/bladders.xacro (robot description, xacro)
@@ -10,5 +10,5 @@
    <xacro:property name="mass" value="1e-2" />
    <xacro:property name="inertia_mom" value="${mass/12}" />
-   <link name="right_bladder">
+<!--    <link name="right_bladder">
      <visual>
        <origin xyz="0 0 0" rpy="0 0 0" />
@@ -53,5 +53,5 @@
         izz="${inertia_mom}"/>
      </inertial>
-   </link>
+   </link> -->
    <link name="big_bladder_link">
      <visual>

File: superchick/headnball.xacro (robot description, xacro)
@@ -14,5 +14,5 @@
        <origin xyz="${0} ${head_y_orig} ${head_z_orig}" rpy="${M_PI/2} 0 ${-M_PI}" />
        <geometry>
-         <mesh filename="package://superchick/meshes/headnball.stl" scale=".001 .001 .001" />
+         <mesh filename="package://superchick/meshes/headnball.dae" scale=".001 .001 .001" />
        </geometry>
        <material name="brown"/>
@@ -21,5 +21,5 @@
      <collision>
        <geometry>
-         <mesh filename="package://superchick/meshes/headnball.stl" scale=".001 .001 .001" />
+         <mesh filename="package://superchick/meshes/headnball.dae" scale=".001 .001 .001" />
        </geometry>
        <origin xyz="${0} ${head_y_orig} ${head_z_orig}" rpy="${M_PI/2} 0 ${-M_PI}" />

File: superchick/superchick.xacro (robot description, xacro)
@@ -6,5 +6,5 @@
    <xacro:property name="damping" value="0.1" />
    <xacro:property name="friction" value="0.2" />
-   <xacro:property name="sim" value="false" />
+   <xacro:property name="sim" value="true" />
   <!-- This file contains the table and bladder descriptions -->
    <xacro:include filename="$(find superchick)/material.xacro" />
@@ -25,5 +25,16 @@
     <origin xyz="${-(table_top_length)/2 + 0.23} 0 ${1e-1/3}" rpy="${0} 0 ${0}" />
   </joint>
-  <joint name="table_to_rightneckbladder" type="fixed">
+  <!-- Actuator Links -->
+  <joint name="bigbladder_to_head" type="continuous">
+    <axis xyz="1 0 0" rpy="0 0 0" />
+    <parent link="big_bladder_link"/>
+    <child link="headnball_link"/>
+    <limit effort="200.0" lower="-0.1016" upper="0.1016" velocity="1.0" />
+    <dynamics damping="${damping}" friction="${friction}" />
+    <safety_controller k_velocity="10" k_position="15" soft_lower_limit="-0.0" soft_upper_limit="0.3" />
+    <origin xyz="${(1e-1/2)+1e-1} ${(table_top_width)/6} 0" rpy="0 0 ${M_PI/2}" />
+  </joint>
+   <!-- Gazebo does not support parallel linkages -->
+<!--   <joint name="table_to_rightneckbladder" type="fixed">
     <parent link="table_top"/>
     <child link="right_bladder"/>
@@ -38,13 +49,4 @@
     <safety_controller k_velocity="10" k_position="15" soft_lower_limit="-0.05" soft_upper_limit="0.05" />
     <origin xyz="${-(table_top_length)/3 + 0.15} -0.12 ${1e-1/3.2}" rpy="${0} 0 ${0}" />
-  </joint>
-  <!-- Actuator Links -->
-  <joint name="bigbladder_to_head" type="continuous">
-    <axis xyz="1 0 0" rpy="0 0 0" />
-    <parent link="big_bladder_link"/>
-    <child link="headnball_link"/>
-    <limit effort="200.0" lower="-0.1016" upper="0.1016" velocity="1.0" />
-    <safety_controller k_velocity="10" k_position="15" soft_lower_limit="-0.0" soft_upper_limit="0.3" />
-    <origin xyz="${(1e-1/2)+1e-1} ${(table_top_width)/6} 0" rpy="0 0 ${M_PI/2}" />
   </joint>
   <joint name="rightbladder_to_neck" type="continuous">
@@ -67,8 +69,10 @@
     <origin xyz="0 0.25 0" rpy="0 0 ${M_PI/2}" />
   </joint>
+ -->
   <joint name="tableTop_to_basePanel" type="fixed">
     <parent link="table_top"/>
     <child link="base_panel"/>
-    <origin xyz="${-(table_top_length)/2 + 0.15} 0 ${1e-1/8}" rpy="${0} 0 ${M_PI/2}" />
+    <!-- <origin xyz="${-(table_top_length)/2 + 0.15} 0 ${1e-1/8}" rpy="${0} 0 ${M_PI/2}"  />-->
+     <origin xyz="${-(table_top_length)/2 + 0.15} 0 ${1e-1/8}" rpy="${0} 0 ${M_PI/2}"/>
   </joint>
   <joint name="vicon_to_world" type="fixed">
@@ -77,7 +81,12 @@
     <origin xyz="-3.5 -2.0 -0.2" rpy="0 0 0" />
   </joint>
+  <joint name="table_to_world" type="fixed">
+    <parent link="world"/>
+    <child link="table_top"/>
+    <origin xyz="-3.5 -2.0 -0.2" rpy="0 0 0" />
+  </joint>
   <transmission name="base_transmission">
      <type>transmission_interface/SimpleTransmission</type>
-     <joint name="joint1">
+     <joint name="bigbladder_to_head">
        <hardwareInterface>EffortJointInterface</hardwareInterface>
      </joint>
@@ -87,5 +96,6 @@
      </actuator>
    </transmission>
-   <transmission name="right_transmission">
+<!--Gazebo does not support parallel linkages
+    <transmission name="right_transmission">
       <type>transmission_interface/SimpleTransmission</type>
       <joint name="rightbladder_to_neck">
@@ -106,4 +116,4 @@
          <mechanicalReduction>1</mechanicalReduction>
        </actuator>
-     </transmission>
+     </transmission> -->
 </robot>

File: superchick/table.xacro (robot description, xacro)
@@ -44,4 +44,8 @@
       </geometry>
     </collision>
+    <inertial>
+      <mass value="1"/>
+        <inertia ixx="0.13" iyy="0.524" izz="0.539" ixy="0" ixz="0" iyz="0" />
+    </inertial>
     <!-- KDL does not support root link inertia mass -->
   </link>

Commit message: updated model with transmission and gazebo controller manager plugin

File: superchick/bladders.xacro (robot description, xacro)
@@ -63,10 +63,10 @@
        <origin xyz="0 0 0" rpy="0 0 0" />
      </visual>
-     <collision>
+<!--      <collision>
        <geometry>
         <box size="${bladder_constant*bladder_length} ${bladder_constant*bladder_width} ${2*bladder_thickness}" />
        </geometry>
        <origin xyz="0 0 0" rpy="0 0 0" />
-     </collision>
+     </collision> -->
      <inertial>
        <mass value="${mass}"/>

File: superchick/superchick.urdf (robot description, URDF)
Before this commit: robot superchick, 8 links, 8 joints
Links:
- link big_bladder_link: geometry visual box size=0.31496 0.31496 0.0508
- link table_top: geometry visual box size=1.524 0.6198 0.0381

File: superchick/superchick.xacro (robot description, xacro)
@@ -26,5 +26,5 @@
   </joint>
   <!-- Actuator Links -->
-  <joint name="bigbladder_to_head" type="continuous">
+  <joint name="bigbladdo_to_head" type="continuous">
     <axis xyz="1 0 0" rpy="0 0 0" />
     <parent link="big_bladder_link"/>
@@ -80,5 +80,5 @@
     <origin xyz="-3.5 -2.0 -0.2" rpy="0 0 0" />
   </joint>
-  <transmission name="base_transmission">
+<!--   <transmission name="base_transmission">
      <type>transmission_interface/SimpleTransmission</type>
      <joint name="bigbladder_to_head">
@@ -89,5 +89,5 @@
        <mechanicalReduction>1</mechanicalReduction>
      </actuator>
-   </transmission>
+   </transmission> -->
 <!--Gazebo does not support parallel linkages
     <transmission name="right_transmission">
@@ -111,3 +111,7 @@
        </actuator>
      </transmission> -->
+<!--      <xacro:include filename="$(find pr2_description)/urdf/sensors/kinect2.urdf.xacro" />
+     <xacro:kinect2_v0 name="head_mount" parent="head_plate_frame" >
+       <origin xyz="-0.137376 0 0.091746" rpy="0 0 0" />
+     </xacro:kinect2_v0> -->
 </robot>

File: superchick/table.xacro (robot description, xacro)
@@ -116,9 +116,9 @@
       <origin xyz="0 0 ${table_leg_height-0.65}" rpy="0 0 0" />
     </visual>
-    <collision>
+<!--     <collision>
       <geometry>
         <box size="${table_top_length} ${table_top_width} ${table_top_thickness}" />
       </geometry>
-    </collision>
+    </collision> -->
     <inertial>
       <mass value="${mass}"/>

Commit message: fake indigo-devel

File: superchick/bladders.xacro (robot description, xacro)
@@ -10,5 +10,5 @@
    <xacro:property name="mass" value="1e-2" />
    <xacro:property name="inertia_mom" value="${mass/12}" />
-<!--    <link name="right_bladder">
+   <link name="right_bladder">
      <visual>
        <origin xyz="0 0 0" rpy="0 0 0" />
@@ -53,5 +53,5 @@
         izz="${inertia_mom}"/>
      </inertial>
-   </link> -->
+   </link>
    <link name="big_bladder_link">
      <visual>
@@ -63,10 +63,10 @@
        <origin xyz="0 0 0" rpy="0 0 0" />
      </visual>
-<!--      <collision>
+     <collision>
        <geometry>
         <box size="${bladder_constant*bladder_length} ${bladder_constant*bladder_width} ${2*bladder_thickness}" />
        </geometry>
        <origin xyz="0 0 0" rpy="0 0 0" />
-     </collision> -->
+     </collision>
      <inertial>
        <mass value="${mass}"/>

File: superchick/headnball.xacro (robot description, xacro)
@@ -19,6 +19,4 @@
        <origin xyz="${0} ${0} ${0}" rpy="${M_PI/2} 0 ${-M_PI}" />
      </visual>
-<!--
-After five days of trying, I realized that adding a collision object to a continuous link causes sdf to produce two separate joints
      <collision>
        <geometry>
@@ -27,11 +25,10 @@
        <origin xyz="${0} ${head_y_orig} ${head_z_orig}" rpy="${M_PI/2} 0 ${-M_PI}" />
      </collision>
- -->
-<!--      <inertial>
+     <inertial>
        <mass value="${mass}"/>
        <inertia ixx="${mass/12}" ixy="0.0" ixz="0.0"
         iyy="${inertia_mom}" iyz="0.0000"
         izz="${inertia_mom}"/>
-     </inertial> -->
+     </inertial>
      <inertial>
        <mass value="1e-1"/>

File: superchick/superchick.xacro (robot description, xacro)
@@ -6,5 +6,5 @@
    <xacro:property name="damping" value="0.1" />
    <xacro:property name="friction" value="0.2" />
-   <xacro:property name="sim" value="true" />
+   <xacro:property name="sim" value="false" />
   <!-- This file contains the table and bladder descriptions -->
    <xacro:include filename="$(find superchick)/material.xacro" />
@@ -12,5 +12,5 @@
    <xacro:include filename="$(find superchick)/bladders.xacro" />
    <xacro:include filename="$(find superchick)/headnball.xacro" />
-   <!-- <xacro:include filename="$(find superchick)/cage.xacro" /> -->
+   <xacro:include filename="$(find superchick)/cage.xacro" />
    <xacro:include filename="$(find superchick)/vicon.xacro" />
    <xacro:if value="${sim == 'true'}">
@@ -36,5 +36,5 @@
   </joint>
    <!-- Gazebo does not support parallel linkages -->
-<!--   <joint name="table_to_rightneckbladder" type="fixed">
+  <joint name="table_to_rightneckbladder" type="fixed">
     <parent link="table_top"/>
     <child link="right_bladder"/>
@@ -69,10 +69,9 @@
     <origin xyz="0 0.25 0" rpy="0 0 ${M_PI/2}" />
   </joint>
- -->
-<!--   <joint name="tableTop_to_basePanel" type="fixed">
+  <joint name="tableTop_to_basePanel" type="fixed">
     <parent link="table_top"/>
     <child link="base_panel"/>
      <origin xyz="${-(table_top_length)/2 + 0.15} 0 ${1e-1/8}" rpy="${0} 0 ${M_PI/2}"  />
-  </joint> -->
+  </joint>
   <joint name="vicon_to_world" type="fixed">
     <parent link="world"/>
@@ -80,5 +79,5 @@
     <origin xyz="-3.5 -2.0 -0.2" rpy="0 0 0" />
   </joint>
-<!--   <transmission name="base_transmission">
+  <transmission name="base_transmission">
      <type>transmission_interface/SimpleTransmission</type>
      <joint name="bigbladder_to_head">
@@ -89,6 +88,6 @@
        <mechanicalReduction>1</mechanicalReduction>
      </actuator>
-   </transmission> -->
-<!--Gazebo does not support parallel linkages
+   </transmission>
+<!-- Gazebo does not support parallel linkages -->
     <transmission name="right_transmission">
       <type>transmission_interface/SimpleTransmission</type>
@@ -110,5 +109,5 @@
          <mechanicalReduction>1</mechanicalReduction>
        </actuator>
-     </transmission> -->
+     </transmission>
 <!--      <xacro:include filename="$(find pr2_description)/urdf/sensors/kinect2.urdf.xacro" />
      <xacro:kinect2_v0 name="head_mount" parent="head_plate_frame" >

File: superchick/table.xacro (robot description, xacro)
@@ -116,9 +116,9 @@
       <origin xyz="0 0 ${table_leg_height-0.65}" rpy="0 0 0" />
     </visual>
-<!--     <collision>
+    <collision>
       <geometry>
         <box size="${table_top_length} ${table_top_width} ${table_top_thickness}" />
       </geometry>
-    </collision> -->
+    </collision>
     <inertial>
       <mass value="${mass}"/>
@@ -147,9 +147,9 @@
       <origin xyz="0 0 ${-table_top_thickness}" rpy="0 0 0" />
     </visual>
-<!--     <collision>
+    <collision>
       <geometry>
         <box size="${table_cover_length} ${table_cover_width/2} ${table_cover_thickness}" />
       </geometry>
-    </collision> -->
+    </collision>
     <inertial>
       <mass value="${mass}"/>
