Commit message: single iab withjout efault ik solvers

File: superchick/bladders.xacro (robot description, xacro)
@@ -10,5 +10,5 @@
    <xacro:property name="mass" value="1e-2" />
    <xacro:property name="inertia_mom" value="${mass/12}" />
-   <link name="right_bladder">
+<!--    <link name="right_bladder">
      <visual>
        <origin xyz="0 0 0" rpy="0 0 0" />
@@ -53,5 +53,5 @@
         izz="${inertia_mom}"/>
      </inertial>
-   </link>
+   </link> -->
    <link name="big_bladder_link">
      <visual>

File: superchick/cage.xacro (robot description, xacro)
@@ -60,5 +60,5 @@
 		<parent link="base_panel"/>
 		<child link="panel_12_oc"/>
-		<origin xyz="0 ${1e-1} ${0.08/2.1}"/>
+		<origin xyz="0 ${distance_panel_12_oc_from_center} ${(panel_thickness/2) + (panel_height/2)}" />
 	</joint>
 	<!-- 9:00 Panel -->

File: superchick/headnball.xacro (robot description, xacro)
@@ -12,14 +12,14 @@
    <link name="headnball_link">
      <visual>
-       <origin xyz="${0} ${0} ${0}" rpy="${M_PI/2} 0 ${-M_PI}" />
+       <origin xyz="${0} ${head_y_orig} ${head_z_orig}" rpy="${M_PI/2} 0 ${-M_PI}" />
        <geometry>
-         <mesh filename="package://superchick/meshes/headnball.dae" scale=".001 .001 .001" />
+         <mesh filename="package://superchick/meshes/headnball.stl" scale=".001 .001 .001" />
        </geometry>
        <material name="brown"/>
-       <origin xyz="${0} ${0} ${0}" rpy="${M_PI/2} 0 ${-M_PI}" />
+       <origin xyz="${0} ${head_y_orig} ${head_z_orig}" rpy="${M_PI/2} 0 ${-M_PI}" />
      </visual>
      <collision>
        <geometry>
-         <mesh filename="package://superchick/meshes/headnball.dae" scale=".001 .001 .001" />
+         <mesh filename="package://superchick/meshes/headnball.stl" scale=".001 .001 .001" />
        </geometry>
        <origin xyz="${0} ${head_y_orig} ${head_z_orig}" rpy="${M_PI/2} 0 ${-M_PI}" />
@@ -31,9 +31,9 @@
         izz="${inertia_mom}"/>
      </inertial>
-     <inertial>
+<!--      <inertial>
        <mass value="1e-1"/>
        <inertia ixx="0.925288" ixy="0.379102" ixz="0.011081"
                 iyy="0.919140" iyz="0.111180" izz="0.993738"/>
-     </inertial>
+     </inertial> -->
    </link>
 </robot>

File: superchick/superchick.urdf (robot description, URDF)
Before this commit: robot superchick, 8 links, 8 joints
Links:
- added link base_panel, mass 0.01; collision box size=0.5842 0.2794 0.0047625; visual box size=0.5842 0.2794 0.0047625
- added link panel_12_oc, mass 0.01; collision box size=0.47 0.200025 0.0047625; visual box size=0.47 0.200025 0.0047625
- added link panel_3_oc, mass 0.01; collision box size=0.231775 0.200025 0.0047625; visual box size=0.231775 0.200025 0.0047625
- added link panel_9_oc, mass 0.01; collision box size=0.231775 0.200025 0.0047625; visual box size=0.231775 0.200025 0.0047625
- link big_bladder_link: geometry collision box size=0.31496 0.31496 0.1016; visual box size=0.31496 0.31496 0.0508
- link headnball_link: mass 1e-1 -> 0.01; geometry collision mesh filename=package://superchick/meshes/headnball.stl scale=.001 .001 .001; visual mesh filename=package://superchick/meshes/headnball.stl scale=.001 .001 .001
- link table_cover: geometry collision box size=1.524 0.2794 0.227; visual box size=1.524 0.2794 0.227
- link table_top: geometry collision box size=1.524 0.6198 0.0381; visual box size=1.524 0.6198 0.0381
- link world: mass 0.1 -> None
Joints:
- added joint 12oc_to_3oc: type fixed, parent panel_12_oc, child panel_3_oc, origin xyz=0.23738125 -0.11350625 0
- added joint 12oc_to_9oc: type fixed, parent panel_12_oc, child panel_9_oc, origin xyz=-0.23738125 -0.11350625 0
- added joint base_panel_to_12oc: type fixed, parent base_panel, child panel_12_oc, origin xyz=0 0.09398 0.10239375
- added joint tableTop_to_basePanel: type fixed, parent table_top, child base_panel, origin xyz=-0.612 0 0.0125 rpy=0.0 0 1.570795
- joint bigbladder_to_head: origin xyz=0.4 0 0.0166666666667 rpy=0 0 1.570795 -> xyz=0.15 0.1033 0 rpy=0 0 1.570795
- joint rightleg_to_tabletop: origin xyz=-0.35 0 0.17  -> xyz=-0.6858 0 0.35 
- joint table_to_big_bladder: origin xyz=-0.254 0 0.0 rpy=0.0 0 0.0 -> xyz=-0.532 0 0.0333333333333 rpy=0.0 0 0.0
- joint tablecover_to_tabletop: origin xyz=0 0 0.0125 rpy=-1.570795 0 0  -> xyz=0 0.2299 -0.18 rpy=-1.570795 0 0 

File: superchick/superchick.xacro (robot description, xacro)
@@ -15,5 +15,5 @@
    <xacro:include filename="$(find superchick)/vicon.xacro" />
    <xacro:if value="${sim == 'true'}">
-    <xacro:include filename="$(find superchick)/superchick.gazebo" />
+    <xacro:include filename="$(find superchick_gazebo)/superchick.gazebo" />
    </xacro:if>
    <!-- table link to bladders -->
@@ -23,20 +23,10 @@
     <limit effort="200.0" lower="0.1016" upper="0.1016" velocity="1.0" />
     <safety_controller k_velocity="10" k_position="15" soft_lower_limit="-0.05" soft_upper_limit="0.05" />
-    <origin xyz="${-(table_top_length)/6} 0 ${0}" rpy="${0} 0 ${0}" />
+    <origin xyz="${-(table_top_length)/2 + 0.23} 0 ${1e-1/3}" rpy="${0} 0 ${0}" />
   </joint>
-  <!-- Actuator Links -->
-  <joint name="bigbladdo_to_head" type="continuous">
-    <axis xyz="1 0 0" rpy="0 0 0" />
-    <parent link="big_bladder_link"/>
-    <child link="headnball_link"/>
-    <limit effort="200.0" lower="-0.1016" upper="0.1016" velocity="1.0" />
-    <dynamics damping="${damping}" friction="${friction}" />
-    <safety_controller k_velocity="10" k_position="15" soft_lower_limit="0.0" soft_upper_limit="0.3" />
-    <origin xyz="${0.4} 0 ${0.1/6}" rpy="0 0 ${M_PI/2}" />
-  </joint>
-   <!-- Gazebo does not support parallel linkages -->
-  <joint name="table_to_rightneckbladder" type="fixed">
+<!--   <joint name="table_to_rightneckbladder" type="fixed">
     <parent link="table_top"/>
     <child link="right_bladder"/>
+    <dynamics damping="0.1"/>
     <limit effort="200.0" lower="0.1016" upper="0.1016" velocity="1.0" />
     <safety_controller k_velocity="10" k_position="15" soft_lower_limit="-0.05" soft_upper_limit="0.05" />
@@ -49,9 +39,20 @@
     <safety_controller k_velocity="10" k_position="15" soft_lower_limit="-0.05" soft_upper_limit="0.05" />
     <origin xyz="${-(table_top_length)/3 + 0.15} -0.12 ${1e-1/3.2}" rpy="${0} 0 ${0}" />
+  </joint> -->
+  <!-- Actuator Links -->
+  <joint name="bigbladder_to_head" type="continuous">
+    <axis xyz="1 0 0" rpy="0 0 0" />
+    <parent link="big_bladder_link"/>
+    <child link="headnball_link"/>
+    <limit effort="200.0" lower="-0.1016" upper="0.1016" velocity="1.0" />
+    <dynamics damping="${damping}" friction="${friction}" />
+    <safety_controller k_velocity="10" k_position="15" soft_lower_limit="0.0" soft_upper_limit="${2*0.3}" />
+    <origin xyz="${(1e-1/2)+1e-1} ${(table_top_width)/6} 0" rpy="0 0 ${M_PI/2}" />
   </joint>
-  <joint name="rightbladder_to_neck" type="continuous">
+<!--   <joint name="rightbladder_to_neck" type="continuous">
     <axis xyz="1 -1 0" rpy="0 0 0" />
-    <parent link="right_bladder"/>
-    <child link="headnball_link"/>
+    <mimic joint="bigbladder_to_head" multiplier="1" offset="0"/>
+    <parent link="headnball_link"/>
+    <child link="right_bladder"/>
     <limit effort="200.0" lower="-0.1016" upper="0.1016" velocity="1.0" />
     <dynamics damping="${damping}" friction="${friction}" />
@@ -61,4 +62,5 @@
   <joint name="leftbladder_to_neck" type="continuous">
     <axis xyz="1 1 0" rpy="0 0 0" />
+    <mimic joint="bigbladder_to_head" multiplier="1" offset="0"/>
     <parent link="left_bladder"/>
     <child link="headnball_link"/>
@@ -68,9 +70,9 @@
     <dynamics damping="${damping}" friction="${friction}" />
     <origin xyz="0 0.25 0" rpy="0 0 ${M_PI/2}" />
-  </joint>
+  </joint>  -->
   <joint name="tableTop_to_basePanel" type="fixed">
     <parent link="table_top"/>
     <child link="base_panel"/>
-     <origin xyz="${-(table_top_length)/2 + 0.15} 0 ${1e-1/8}" rpy="${0} 0 ${M_PI/2}"  />
+    <origin xyz="${-(table_top_length)/2 + 0.15} 0 ${1e-1/8}" rpy="${0} 0 ${M_PI/2}" />
   </joint>
   <joint name="vicon_to_world" type="fixed">
@@ -89,6 +91,5 @@
      </actuator>
    </transmission>
-<!-- Gazebo does not support parallel linkages -->
-    <transmission name="right_transmission">
+<!--    <transmission name="right_transmission">
       <type>transmission_interface/SimpleTransmission</type>
       <joint name="rightbladder_to_neck">
@@ -109,8 +110,4 @@
          <mechanicalReduction>1</mechanicalReduction>
        </actuator>
-     </transmission>
-<!--      <xacro:include filename="$(find pr2_description)/urdf/sensors/kinect2.urdf.xacro" />
-     <xacro:kinect2_v0 name="head_mount" parent="head_plate_frame" >
-       <origin xyz="-0.137376 0 0.091746" rpy="0 0 0" />
-     </xacro:kinect2_v0> -->
+     </transmission> -->
 </robot>

File: superchick/table.xacro (robot description, xacro)
@@ -44,8 +44,4 @@
       </geometry>
     </collision>
-    <inertial>
-      <mass value="0.1"/>
-        <inertia ixx="0.13" iyy="0.524" izz="0.539" ixy="0" ixz="0" iyz="0" />
-    </inertial>
     <!-- KDL does not support root link inertia mass -->
   </link>
@@ -131,5 +127,5 @@
     <parent link="right_leg"/>
     <child link="table_top" />
-    <origin xyz="-0.35 0 0.17 " />
+    <origin xyz="${-(table_top_length/2)+0.0762} 0 0.35 " />
   </joint>
   <joint name="leftleg_to_tabletop" type="fixed">
@@ -142,5 +138,5 @@
       <origin xyz="0 0 ${-table_top_thickness}" rpy="0 0 0" />
       <geometry>
-        <box size="${table_cover_length} ${table_cover_width/2} ${table_cover_thickness}" />
+        <box size="${table_cover_length} ${table_cover_width} ${table_cover_thickness}" />
       </geometry>
       <material name="table_cover_color"/>
@@ -149,5 +145,5 @@
     <collision>
       <geometry>
-        <box size="${table_cover_length} ${table_cover_width/2} ${table_cover_thickness}" />
+        <box size="${table_cover_length} ${table_cover_width} ${table_cover_thickness}" />
       </geometry>
     </collision>
@@ -162,5 +158,5 @@
     <parent link="table_top"/>
     <child link="table_cover"/>
-    <origin xyz="0 0 ${0.05/4}" rpy="${-M_PI/2} 0 0 "/>
+    <origin xyz="0 ${(table_top_width/2)-0.08} -0.18" rpy="${-M_PI/2} 0 0 "/>
   </joint>
 </robot>
